File: pcb/pHMeter/pHMeter.kicad_pcb (KiCad board)
At the start: 2 copper layers, 124 parts, among them J1 Conn_02x03_Odd_Even, J2 Conn_Coaxial_Power, J3 Conn_Coaxial_Power, J4 Conn_Coaxial_Power, J5 RJ12, J6 RJ12, J7 SJ, J8 SJ, Q1 BSP75, Q2 BSP75, Q3 FDN340P, U1 TLV6004PW, U2 TLV6004PW, U3 ATMEGA32U4-AU, U4 ACT4088, U5 AP63203WU-7, U6 HX711, U7 SST25VF064C, X1 MINI-USB-SCHIELD-32005-201, Y1 Crystal

Commit message: update pcb
Parts:
- U7: value SST25VF064C -> SST26VF064B; footprint Package_SO:SOIC-16W_7.5x10.3mm_P1.27mm -> Package_SO:SOIJ-8_5.3x5.3mm_P1.27mm
- moved J6 195.2 mm to (223.3, 132.6)
- moved R15 170.9 mm to (245.9, 135.6), turned to 90 degrees
- moved R36 146.9 mm to (228.6, 105.9)
- moved C13 146.9 mm to (254.8, 112.3)
- moved C14 146.9 mm to (254.8, 118.1)
- moved C15 146.9 mm to (250.2, 122.7)
- moved C17 146.9 mm to (239.8, 105.7)
- moved C18 146.9 mm to (235.5, 123.7)
- moved J7 146.9 mm to (254.8, 122.5)
- moved JP5 146.9 mm to (225.3, 110.2)
- moved R34 146.9 mm to (246.9, 122.7)
- moved R35 146.9 mm to (245.6, 115.1)
- moved U3 146.9 mm to (235.5, 114.8)
- moved Y1 146.9 mm to (250.2, 115.2)
- moved C16 146.9 mm to (226.1, 117.3)
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Other:
- board outline added: 99.1 x 85.1 mm

Commit message: pcb phMeter
Parts:
- moved R20 137.2 mm to (229.6, 102.5), turned to 180 degrees
- moved JP2 133.3 mm to (200.4, 109.5), turned to 270 degrees
- moved JP1 127.4 mm to (200.4, 105.4), turned to 270 degrees
- moved D8 95.3 mm to (226.3, 101.6), turned to 270 degrees
- moved D16 85.2 mm to (216.7, 114.0)
- moved U4 79.1 mm to (212.3, 106.2)
- moved D15 79.1 mm to (212.6, 114.0), turned to 180 degrees
- moved D5 78.2 mm to (136.8, 86.4)
- moved R40 74.7 mm to (219.7, 111.0), turned to 270 degrees
- moved C23 73.9 mm to (217.4, 103.6)
- moved R37 72.5 mm to (215.4, 110.5)
- moved D14 69.9 mm to (207.1, 102.6), turned to 180 degrees
- moved R38 68.7 mm to (216.4, 107.5), turned to 270 degrees
- moved C20 66.4 mm to (207.5, 108.7), turned to 180 degrees
- moved R39 65.0 mm to (208.3, 113.0), turned to 270 degrees
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Connections:
- U4 pad 3: Net-(U4-Pad3) -> VDD
Other:
- board text added: "3.3 V Buck"
- board text added: "Test 12 V"
- board text added: "Test 3.3 V"
- board text added: "uC"

Commit message: Update pHMeter pcb
Parts:
- TP1, TP2: footprint TestPoint:TestPoint_Pad_D1.5mm -> TestPoint:TestPoint_Pad_D1.0mm
- U2: footprint Package_DFN_QFN:Texas_S-PX2QFN-14 -> Package_SO:TSSOP-14_4.4x5mm_P0.65mm
- moved C3 146.3 mm to (217.0, 35.6), turned to 180 degrees
- moved R24 142.4 mm to (267.7, 114.3), turned to 180 degrees
- moved J4 137.0 mm to (191.3, 126.5)
- moved R42 136.8 mm to (270.8, 125.2)
- moved D6 136.0 mm to (164.8, 32.8)
- moved D1 134.9 mm to (135.3, 36.8)
- moved J1 134.2 mm to (242.8, 123.3)
- moved D2 132.1 mm to (135.3, 34.3), turned to 180 degrees
- moved R3 131.7 mm to (216.9, 31.0), turned to 180 degrees
- moved C31 129.6 mm to (272.0, 114.3)
- moved D11 129.0 mm to (262.9, 112.0)
- moved R4 125.2 mm to (216.9, 33.3), turned to 180 degrees
- moved C9 119.3 mm to (220.2, 43.1), turned to 270 degrees
- moved R8 112.7 mm to (163.3, 27.2)
- moved TP1 112.5 mm to (122.9, 44.7)
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Connections:
- D11 pad 1: D10 -> TX
- DS1 pad 14: A4 -> D10
- R44 pad 2: D10 -> TX
- U1 pad 1: Net-(C5-Pad2) -> Net-(J3-Pad2)
- U1 pad 2: Net-(D1-Pad1) -> Net-(J3-Pad2)
- U1 pad 3: Net-(C2-Pad2) -> Net-(C3-Pad1)
- U2 pad 1: Net-(J3-Pad2) -> Net-(C5-Pad2)
- U2 pad 2: Net-(J3-Pad2) -> Net-(D1-Pad1)
- U2 pad 3: Net-(C3-Pad1) -> Net-(C2-Pad2)
Other:
- board text added: "Flash"

Commit message: Update pHMeter pcb
Parts:
- moved Q1 222.1 mm to (266.8, 86.3)
- moved JP4 213.8 mm to (274.3, 83.8)
- moved J8 202.6 mm to (238.3, 24.9), turned to 270 degrees
- moved C27 195.8 mm to (227.6, 21.6), turned to 90 degrees
- moved C28 193.2 mm to (225.0, 28.4), turned to 270 degrees
- moved C26 193.1 mm to (224.0, 24.1), turned to 180 degrees
- moved D3 191.9 mm to (245.2, 138.9), turned to 180 degrees
- moved JP3 191.5 mm to (274.3, 94.5)
- moved Q2 191.2 mm to (266.8, 96.3)
- moved D4 190.2 mm to (249.4, 137.3), turned to 90 degrees
- moved C29 184.6 mm to (221.5, 28.4), turned to 270 degrees
- moved R26 172.9 mm to (260.4, 85.3), turned to 270 degrees
- moved C11 164.7 mm to (262.1, 137.9), turned to 180 degrees
- moved R27 158.7 mm to (260.2, 95.0), turned to 270 degrees
- moved R21 153.6 mm to (249.9, 89.9), turned to 270 degrees
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Connections:
- U1 pad 12: Net-(R18-Pad2) -> (no net)
- U1 pad 13: Net-(R19-Pad2) -> (no net)
- U1 pad 14: A+ -> (no net)
- U2 pad 12: (no net) -> Net-(R18-Pad2)
- U2 pad 13: (no net) -> Net-(R19-Pad2)
- U2 pad 14: (no net) -> A+
Other:
- board text added: "Foods"
