File: pcb/pHMeter/pHMeter.kicad_pcb (KiCad board)
At the start: 2 copper layers, 99.1 x 85.1 mm, 116 parts, among them J1 Conn_02x03_Odd_Even, J2 Conn_Coaxial_Power, J3 Conn_Coaxial_Power, J4 Conn_Coaxial_Power, J5 RJ12, J6 RJ12, J7 SJ, J8 SJ, Q1 BSP75, Q2 BSP75, Q3 FDN340P, U1 TLV6004PW, U2 TLV6004PW, U3 ATMEGA32U4-AU, U5 AP63203WU-7, U6 HX711, U7 SST26VF064B, X1 MINI-USB-SCHIELD-32005-201, Y1 Crystal

Commit message: Update pcb pHmeter and doc
Parts:
- removed JP5: M02JST-PTH-2, Connector_PinHeader_2.54mm:PinHeader_1x02_P2.54mm_Vertical
- removed Q3: FDN340P, Package_TO_SOT_SMD:SOT-23
- removed R29: 1k, Resistor_SMD:R_0805_2012Metric_Pad1.15x1.40mm_HandSolder
- removed R30: 220k, Resistor_SMD:R_0805_2012Metric_Pad1.15x1.40mm_HandSolder
- added SW1: Rotary_Encoder_Switch, Rotary_Encoder:RotaryEncoder_Alps_EC11E-Switch_Vertical_H20mm, F.Cu at (229.4, 84.8)
- J5, J6: footprint Connector_RJ:RJ12_Amphenol_54601 -> Connector_RJ:RJ25_Wayconn_MJEA-660X1_Horizontal
- Q1, Q2: value BSP75 -> ZXMS6004; footprint Package_TO_SOT_SMD:SOT-223-3_TabPin2 -> Package_TO_SOT_SMD:SOT-23
- moved DS1 166.0 mm to (182.9, 139.3), turned to 90 degrees
- moved R31 121.4 mm to (186.9, 103.6), turned to 180 degrees
- moved R32 111.6 mm to (229.4, 75.4), turned to 270 degrees
- moved RV1 109.2 mm to (226.1, 76.5), turned to 90 degrees
- moved R33 107.6 mm to (217.9, 82.0), turned to 270 degrees
- moved D7 86.6 mm to (272.9, 131.9), turned to 180 degrees
- moved R16 78.1 mm to (268.7, 131.8), turned to 0 degrees
- moved J4 68.4 mm to (257.0, 135.9), turned to 90 degrees
- moved C5 66.8 mm to (212.4, 104.4)
- moved C8 66.8 mm to (208.4, 94.7)
- moved D1 66.8 mm to (213.0, 97.0)
- moved R12 66.8 mm to (199.4, 98.6)
- moved R5 66.8 mm to (212.6, 106.7)
- moved R9 66.8 mm to (208.3, 97.0)
- moved C10 66.8 mm to (212.5, 101.9)
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Connections:
- DS1 pad 2: Net-(DS1-Pad2) -> D13
Other:
- board size 99.1 x 85.1 mm -> 100 x 82.5 mm
- board text added: "12 V"
- board text added: "3.3 V"
- board text added: "Conductometer"
- board text added: "PH"
- board text removed: "3.3 V Buck"

Commit message: New Li-Po
Parts:
- added U4: LTC4089EDJCPBF, pHMeter:QFN-22-1EP_6x3mm_P0.5mm_EP1.65x5.35_ThermalVias, F.Cu at (153.4, 120.7)
- moved C11 45.2 mm to (221.2, 135.7)
- moved R14 45.2 mm to (224.8, 135.6)
- moved R15 45.2 mm to (227.1, 135.6)
- moved X1 45.2 mm to (226.3, 143.5)
- moved J4 13.7 mm to (270.8, 135.9)
- moved TP2 13.7 mm to (263.1, 133.9)
- moved J5 13.7 mm to (243.4, 138.7)
- moved J6 13.7 mm to (259.9, 138.7)
- moved R25 4.59 mm to (236.5, 133.3)
- moved R28 2.34 mm to (235.7, 131.1)
- moved C32 0.51 mm to (222.4, 128.3)

Commit message: update pcb pHMeter
Parts:
- removed C32: 100u, Capacitor_SMD:CP_Elec_6.3x7.7
- removed TP2: TestPoint, TestPoint:TestPoint_Pad_D1.0mm
- added C20: 10u, Capacitor_SMD:C_0805_2012Metric_Pad1.15x1.40mm_HandSolder, F.Cu at (309.8, 127.9)
- added C21: 10u, Capacitor_SMD:C_0805_2012Metric_Pad1.15x1.40mm_HandSolder, F.Cu at (304.2, 120.4)
- added C23: 10u, Capacitor_SMD:C_0805_2012Metric_Pad1.15x1.40mm_HandSolder, F.Cu at (299.4, 123.0)
- added C33: 100n, Capacitor_SMD:C_0805_2012Metric_Pad1.15x1.40mm_HandSolder, F.Cu at (308.9, 112.7)
- added D14: D_Schottky, Diode_SMD:D_SOD-123, F.Cu at (295.2, 127.3)
- added D17: LED, LED_SMD:LED_0805_2012Metric_Pad1.15x1.40mm_HandSolder, F.Cu at (299.4, 120.0)
- added D18: LED, LED_SMD:LED_0805_2012Metric_Pad1.15x1.40mm_HandSolder, F.Cu at (304.2, 117.4)
- added D19: TX, LED_SMD:LED_0805_2012Metric_Pad1.15x1.40mm_HandSolder, F.Cu at (233.9, 130.0)
- added D20: TX, LED_SMD:LED_0805_2012Metric_Pad1.15x1.40mm_HandSolder, F.Cu at (220.2, 130.0)
- added H1: MountingHole, MountingHole:MountingHole_3.2mm_M3, F.Cu at (183.6, 144.3)
- added H2: MountingHole, MountingHole:MountingHole_3.2mm_M3, F.Cu at (275.1, 144.3)
- added H3: MountingHole, MountingHole:MountingHole_3.2mm_M3, F.Cu at (183.6, 65.8)
- added H4: MountingHole, MountingHole:MountingHole_3.2mm_M3, F.Cu at (275.1, 65.8)
- added JP5: Bat, Connector_PinHeader_2.54mm:PinHeader_1x02_P2.54mm_Vertical, F.Cu at (294.7, 113.6)
- added JP6: IO3, Connector_PinHeader_2.54mm:PinHeader_1x02_P2.54mm_Vertical, F.Cu at (294.7, 120.8)
- added JP7: IO4, Connector_PinHeader_2.54mm:PinHeader_1x02_P2.54mm_Vertical, F.Cu at (299.3, 113.6)
- added Q3: DMP1045, Package_TO_SOT_SMD:SOT-23, F.Cu at (309.8, 124.2)
- added Q4: ZXMS6004, Package_TO_SOT_SMD:SOT-23, F.Cu at (323.0, 113.5)
- added Q5: ZXMS6004, Package_TO_SOT_SMD:SOT-23, F.Cu at (313.5, 119.4)
- added R29: 10k, Resistor_SMD:R_0805_2012Metric_Pad1.15x1.40mm_HandSolder, F.Cu at (300.5, 125.9)
- added R30: 10k, Resistor_SMD:R_0805_2012Metric_Pad1.15x1.40mm_HandSolder, F.Cu at (313.6, 112.7)
- added R37: 10k, Resistor_SMD:R_0805_2012Metric_Pad1.15x1.40mm_HandSolder, F.Cu at (309.0, 115.7)
- added R38: 1M, Resistor_SMD:R_0805_2012Metric_Pad1.15x1.40mm_HandSolder, F.Cu at (308.9, 120.4)
- added R45: 1M, Resistor_SMD:R_0805_2012Metric_Pad1.15x1.40mm_HandSolder, F.Cu at (305.2, 123.4)
- added R46: 100k, Resistor_SMD:R_0805_2012Metric_Pad1.15x1.40mm_HandSolder, F.Cu at (313.7, 115.7)
- added R47: 10k, Resistor_SMD:R_0805_2012Metric_Pad1.15x1.40mm_HandSolder, F.Cu at (318.4, 112.7)
- added R48: 10k, Resistor_SMD:R_0805_2012Metric_Pad1.15x1.40mm_HandSolder, F.Cu at (305.2, 126.3)
- added R49: 1k, Resistor_SMD:R_0805_2012Metric_Pad1.15x1.40mm_HandSolder, F.Cu at (239.8, 130.0)
- added R50: 1k, Resistor_SMD:R_0805_2012Metric_Pad1.15x1.40mm_HandSolder, F.Cu at (225.6, 130.0)
- added R51: 4.7k, Resistor_SMD:R_0805_2012Metric_Pad1.15x1.40mm_HandSolder, F.Cu at (237.2, 130.1)
- added R52: 4.7k, Resistor_SMD:R_0805_2012Metric_Pad1.15x1.40mm_HandSolder, F.Cu at (223.3, 130.1)
- added R53: 100, Resistor_SMD:R_0805_2012Metric_Pad1.15x1.40mm_HandSolder, F.Cu at (229.4, 130.1)
- added R54: 100, Resistor_SMD:R_0805_2012Metric_Pad1.15x1.40mm_HandSolder, F.Cu at (215.6, 130.0)
- added R55: 1k, Resistor_SMD:R_0805_2012Metric_Pad1.15x1.40mm_HandSolder, F.Cu at (231.6, 130.1)
- added R56: 1k, Resistor_SMD:R_0805_2012Metric_Pad1.15x1.40mm_HandSolder, F.Cu at (217.9, 130.1)
- added U9: MCP73811T, Package_TO_SOT_SMD:SOT-23-5, F.Cu at (304.1, 113.6)
- C1, C10, C11, C12, C2, C3, C4, C5, C6, C7, C8, C9: footprint Capacitor_SMD:C_0805_2012Metric -> Capacitor_SMD:C_0805_2012Metric_Pad1.15x1.40mm_HandSolder
- DS1, SW1: moved to B.Cu
- J4: value Conn_Coaxial_Power -> AudioJack3_SwitchTR; footprint Connector_BarrelJack:BarrelJack_Horizontal -> Connector_Audio:Jack_3.5mm_Ledino_KB3SPRS_Horizontal
- J5: footprint Connector_RJ:RJ25_Wayconn_MJEA-660X1_Horizontal -> pHMeter:E5566-Q0LK22-L
- J6: value RJ12 -> AudioJack3_SwitchTR; footprint Connector_RJ:RJ25_Wayconn_MJEA-660X1_Horizontal -> Connector_Audio:Jack_3.5mm_Ledino_KB3SPRS_Horizontal
- U4: value LTC4089EDJCPBF -> MCP1703A; footprint pHMeter:QFN-22-1EP_6x3mm_P0.5mm_EP1.65x5.35_ThermalVias -> Package_TO_SOT_SMD:SOT-23
- moved R27 228.9 mm to (41.0, 139.2)
- moved D12 228.9 mm to (40.0, 142.8)
- moved D13 228.9 mm to (40.1, 134.9)
- moved JP3 228.9 mm to (49.5, 139.4)
- moved JP4 228.9 mm to (49.5, 131.8)
- moved R26 228.9 mm to (41.1, 131.6)
- moved Q1 228.9 mm to (45.3, 132.6)
- moved Q2 228.9 mm to (45.3, 140.5)
- moved J3 175.3 mm to (94.2, 86.4), turned to 0 degrees
- moved R11 170.7 mm to (85.9, 64.8), turned to 180 degrees
- moved U1 170.0 mm to (85.9, 68.8), turned to 180 degrees
- moved U4 165.0 mm to (318.3, 116.5)
- moved C9 164.3 mm to (89.2, 64.1), turned to 90 degrees
- moved D9 161.0 mm to (101.6, 64.0), turned to 270 degrees
- moved R21 159.1 mm to (101.6, 69.1), turned to 90 degrees
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Connections:
- C19 pad 1: VDD -> VBAT
- C6 pad 1: 12V -> Net-(C6-Pad1)
- C7 pad 1: 12V -> Net-(C6-Pad1)
- D5 pad 2: 12V -> Net-(C6-Pad1)
- R39 pad 1: VDD -> VBAT
- U4 pad 1: Net-(U4-Pad1) -> GND
- U4 pad 2: Net-(U4-Pad2) -> Net-(C6-Pad1)
- U4 pad 3: Net-(U4-Pad3) -> 12V
- U5 pad 2: VDD -> VBAT
- U5 pad 3: VDD -> VBAT
Other:
- board size 100 x 82.5 mm -> 100 x 87 mm
- board text added: "I2C"
- board text added: "One Wire"
- board text added: "USB"
