File: pcb/pHMeter/_autosave-pHMeter.kicad_pcb (KiCad board)
At the start: 2 copper layers, 99.1 x 85.1 mm, 116 parts, among them J1 Conn_02x03_Odd_Even, J2 Conn_Coaxial_Power, J3 Conn_Coaxial_Power, J4 Conn_Coaxial_Power, J5 RJ12, J6 RJ12, J7 SJ, J8 SJ, Q1 BSP75, Q2 BSP75, Q3 FDN340P, U1 TLV6004PW, U2 TLV6004PW, U3 ATMEGA32U4-AU, U5 AP63203WU-7, U6 HX711, U7 SST26VF064B, X1 MINI-USB-SCHIELD-32005-201, Y1 Crystal

Commit message: Update sch & pcb
Parts:
- removed Q3: FDN340P, Package_TO_SOT_SMD:SOT-23
- removed R29: 1k, Resistor_SMD:R_0805_2012Metric_Pad1.15x1.40mm_HandSolder
- removed R30: 220k, Resistor_SMD:R_0805_2012Metric_Pad1.15x1.40mm_HandSolder
Connections:
- DS1 pad 2: Net-(DS1-Pad2) -> D13
