File: pcb/pHMeter/3.sch (KiCad schematic (older format))
At the start: 18 parts, among them U4 ACT4088, U5 AP63203WU-7

Commit message: pcb and footprints
Parts:
- renumbered D7 to D14, D8 to D15, D9 to D16, R32 to R37, R33 to R38, R34 to R39, R35 to R40
Changed lines of the file:
@@
 $EndComp
 $Comp
-L Device:R R33
+L Device:R R38
 U 1 1 5E004CDB
 P 5125 4350
-F 0 "R33" V 5225 4400 50  0000 C CNN
+F 0 "R38" V 5225 4400 50  0000 C CNN
 F 1 "49.9k" V 5025 4400 50  0000 C CNN
 F 2 "Resistor_SMD:R_0805_2012Metric_Pad1.15x1.40mm_HandSolder" V 5055 4350 50  0001 C CNN
@@
 $EndComp
 $Comp
-L Device:R R32
+L Device:R R37
 U 1 1 5E004CE1
 P 4775 4600
-F 0 "R32" H 4705 4554 50  0000 R CNN
+F 0 "R37" H 4705 4554 50  0000 R CNN
 F 1 "16.23k" H 4705 4645 50  0000 R CNN
 F 2 "Resistor_SMD:R_0805_2012Metric_Pad1.15x1.40mm_HandSolder" V 4705 4600 50  0001 C CNN
@@
 	5575 3950 6175 3950
 $Comp
-L Device:D D7
+L Device:D D14
 U 1 1 5E004D28
 P 4775 4100
-F 0 "D7" V 4729 4179 50  0000 L CNN
+F 0 "D14" V 4729 4179 50  0000 L CNN
 F 1 "B240A" V 4820 4179 50  0000 L CNN
 F 2 "Diode_SMD:D_SOD-123" H 4775 4100 50  0001 C CNN
@@
 AR Path="/5E1D0FCF" Ref="R?"  Part="1"
 AR Path="/5E0005EE/5E1D0FCF" Ref="R?"  Part="1"
-AR Path="/5ED0DFF6/5E1D0FCF" Ref="R34"  Part="1"
-F 0 "R34" V 8250 3625 50  0000 C CNN
+AR Path="/5ED0DFF6/5E1D0FCF" Ref="R39"  Part="1"
+F 0 "R39" V 8250 3625 50  0000 C CNN
 F 1 "10k" V 8325 3625 50  0000 C CNN
 F 2 "Resistor_SMD:R_0805_2012Metric_Pad1.15x1.40mm_HandSolder" V 8255 3625 50  0001 C CNN
@@
 AR Path="/5E1D0FDF" Ref="R?"  Part="1"
 AR Path="/5E0005EE/5E1D0FDF" Ref="R?"  Part="1"
-AR Path="/5ED0DFF6/5E1D0FDF" Ref="R35"  Part="1"
-F 0 "R35" V 8250 4225 50  0000 C CNN
+AR Path="/5ED0DFF6/5E1D0FDF" Ref="R40"  Part="1"
+F 0 "R40" V 8250 4225 50  0000 C CNN
 F 1 "1k" V 8325 4225 50  0000 C CNN
 F 2 "Resistor_SMD:R_0805_2012Metric_Pad1.15x1.40mm_HandSolder" V 8255 4225 50  0001 C CNN
@@
 Connection ~ 3775 3700
 $Comp
-L Device:LED D8
+L Device:LED D15
 U 1 1 5E883301
 P 7425 3625
-F 0 "D8" H 7425 3550 50  0000 C CNN
+F 0 "D15" H 7425 3550 50  0000 C CNN
 F 1 "RED" H 7425 3725 50  0000 C CNN
 F 2 "LED_SMD:LED_0805_2012Metric_Pad1.15x1.40mm_HandSolder" H 7425 3625 50  0001 C CNN
@@
 $EndComp
 $Comp
-L Device:LED D9
+L Device:LED D16
 U 1 1 5E886D2D
 P 7425 4225
-F 0 "D9" H 7425 4150 50  0000 C CNN
+F 0 "D16" H 7425 4150 50  0000 C CNN
 F 1 "RED" H 7425 4325 50  0000 C CNN
 F 2 "LED_SMD:LED_0805_2012Metric_Pad1.15x1.40mm_HandSolder" H 7425 4225 50  0001 C CNN

Commit message: pcb phMeter
Connections:
- net VIN: now also U4.3 (EN)
- no-connect marks 2 -> 1
Other:
- moved on the sheet: C19
Changed lines of the file:
@@
 F 3 "~" H 3775 3900 50  0001 C CNN
 	1    3775 3900
-	1    0    0    -1
+	-1   0    0    -1
 $EndComp
 Wire Wire Line
@@
 	0    1    1    0
 $EndComp
-NoConn ~ 4025 4150
 Text Notes 6700 3425 0    118  ~ 0
 Power LEDS
@@
 	5575 4300 5575 4500
 Wire Wire Line
-	4025 3700 3775 3700
+	4025 3700 3975 3700
 Connection ~ 3775 3700
 $Comp
@@
 L Device:C C19
 U 1 1 5EDC3622
-P 3650 6000
-F 0 "C19" H 3765 6046 50  0000 L CNN
-F 1 "10u" H 3765 5955 50  0000 L CNN
-F 2 "Capacitor_SMD:C_0805_2012Metric_Pad1.15x1.40mm_HandSolder" H 3688 5850 50  0001 C CNN
-F 3 "~" H 3650 6000 50  0001 C CNN
-	1    3650 6000
+P 3625 6000
+F 0 "C19" H 3740 6046 50  0000 L CNN
+F 1 "10u" H 3740 5955 50  0000 L CNN
+F 2 "Capacitor_SMD:C_0805_2012Metric_Pad1.15x1.40mm_HandSolder" H 3663 5850 50  0001 C CNN
+F 3 "~" H 3625 6000 50  0001 C CNN
+	1    3625 6000
 	1    0    0    -1
 $EndComp
@@
 	3900 5800 3950 5800
 Wire Wire Line
-	3900 5800 3650 5800
-Wire Wire Line
-	3650 5800 3650 5850
-Connection ~ 3900 5800
-Wire Wire Line
-	3650 5800 3600 5800
-Connection ~ 3650 5800
-Wire Wire Line
-	3650 6225 3650 6150
+	3625 5800 3625 5850
+Wire Wire Line
+	3625 5800 3575 5800
+Connection ~ 3625 5800
+Wire Wire Line
+	3625 6225 3625 6150
 Wire Wire Line
 	4350 6200 4350 6275
-Text HLabel 3600 5800 0    50   Input ~ 0
+Text HLabel 3575 5800 0    50   Input ~ 0
 VIN
-Text HLabel 3650 6225 0    50   Input ~ 0
+Text HLabel 3625 6225 0    50   Input ~ 0
 GND
 Text HLabel 4350 6275 0    50   Input ~ 0
@@
 	1    0    0    -1
 $EndComp
+Wire Wire Line
+	4025 4150 3975 4150
+Wire Wire Line
+	3975 4150 3975 3700
+Connection ~ 3975 3700
+Wire Wire Line
+	3975 3700 3775 3700
+Wire Wire Line
+	3625 5800 3900 5800
+Connection ~ 3900 5800
 $EndSCHEMATC

Commit message: Update sch & pcb
Parts:
- removed C20: 10µF, Capacitor_SMD:C_0805_2012Metric_Pad1.15x1.40mm_HandSolder, symbol Device:C
- removed C21: 22nF, Capacitor_SMD:C_0805_2012Metric_Pad1.15x1.40mm_HandSolder, symbol Device:C
- removed C23: 22µF, Capacitor_SMD:C_0805_2012Metric_Pad1.15x1.40mm_HandSolder, symbol Device:C
- removed D14: B240A, Diode_SMD:D_SOD-123, symbol Device:D
- removed L1: 4.7µH, Inductor_SMD:L_0805_2012Metric_Pad1.15x1.40mm_HandSolder, symbol Device:L
- removed R37: 16.23k, Resistor_SMD:R_0805_2012Metric_Pad1.15x1.40mm_HandSolder, symbol Device:R
- removed R38: 49.9k, Resistor_SMD:R_0805_2012Metric_Pad1.15x1.40mm_HandSolder, symbol Device:R
- removed U4: ACT4088, Package_TO_SOT_SMD:SOT-23-6_Handsoldering, symbol ACT4088:ACT4088
Other:
- note added: "3.3 V Buck"
- note added: "The inductor’s DC resistance should be less than 100mΩ.\n \nThe input capacitor, electrolytic, or ceramics with low ESR\nshould be used."
- note removed: "3.3v: 16.23k\n5v: 9.64k"
- note removed: "LDPW12\n"
- note removed: "LDPW3\n"
- note removed: "The inductor’s DC resistance should be less than 100mΩ.\n \nThe input capacitor, electrolytic, or ceramics with low ESR should be used."
- moved on the sheet: C19, C22, C24, C25, D15, D16, L2, R39, R40, U5
