File: pcb/pHMeter/pH.sch (KiCad schematic (older format))
At the start: 9 parts, among them J3 Conn_Coaxial_Power, U1 TLV6004PW

Commit message: update pcb pHMeter
Parts:
- C1, C3, C9: footprint Capacitor_SMD:C_0805_2012Metric -> Capacitor_SMD:C_0805_2012Metric_Pad1.15x1.40mm_HandSolder
Changed lines of the file:
@@
 F 0 "C3" H 4665 4546 50  0000 L CNN
 F 1 "100n" H 4665 4455 50  0000 L CNN
-F 2 "Capacitor_SMD:C_0805_2012Metric" H 4588 4350 50  0001 C CNN
+F 2 "Capacitor_SMD:C_0805_2012Metric_Pad1.15x1.40mm_HandSolder" H 4588 4350 50  0001 C CNN
 F 3 "~" H 4550 4500 50  0001 C CNN
 	1    4550 4500
@@
 F 0 "C9" H 7915 4446 50  0000 L CNN
 F 1 "22u" H 7915 4355 50  0000 L CNN
-F 2 "Capacitor_SMD:C_0805_2012Metric" H 7838 4250 50  0001 C CNN
+F 2 "Capacitor_SMD:C_0805_2012Metric_Pad1.15x1.40mm_HandSolder" H 7838 4250 50  0001 C CNN
 F 3 "~" H 7800 4400 50  0001 C CNN
 	1    7800 4400
@@
 F 0 "C1" H 3965 4146 50  0000 L CNN
 F 1 "100n" H 3965 4055 50  0000 L CNN
-F 2 "Capacitor_SMD:C_0805_2012Metric" H 3888 3950 50  0001 C CNN
+F 2 "Capacitor_SMD:C_0805_2012Metric_Pad1.15x1.40mm_HandSolder" H 3888 3950 50  0001 C CNN
 F 3 "~" H 3850 4100 50  0001 C CNN
 	1    3850 4100
