File: pcb/main/3.sch (KiCad schematic (older format))
At the start: 12 parts, among them U3 ACT4088

Commit message: feat: add 2 IO, 1 one wire, fan and 3 stepper output. Closes: #20 #11 #9 #4
Parts:
- D11, D13: value RED -> GREEN
Changed lines of the file:
@@
 P 7425 3625
 F 0 "D11" H 7425 3550 50  0000 C CNN
-F 1 "RED" H 7425 3725 50  0000 C CNN
+F 1 "GREEN" H 7425 3725 50  0000 C CNN
 F 2 "LED_SMD:LED_0805_2012Metric_Pad1.15x1.40mm_HandSolder" H 7425 3625 50  0001 C CNN
 F 3 "~" H 7425 3625 50  0001 C CNN
@@
 P 7425 4225
 F 0 "D13" H 7425 4150 50  0000 C CNN
-F 1 "RED" H 7425 4325 50  0000 C CNN
+F 1 "GREEN" H 7425 4325 50  0000 C CNN
 F 2 "LED_SMD:LED_0805_2012Metric_Pad1.15x1.40mm_HandSolder" H 7425 4225 50  0001 C CNN
 F 3 "~" H 7425 4225 50  0001 C CNN
