File: pcb/main/Load cell 24bits ADC.sch (KiCad schematic (older format))
At the start: 17 parts, among them J9 SJ, Q4 TRANSISTOR_PNPMMBT4403, U4 HX711HX711

Commit message: fix: update arduino code
Connections:
- net A4 renamed DATA
- net A5 renamed CLK
Changed lines of the file:
@@
 GND
 Text HLabel 7375 3600 2    59   Input ~ 0
-A4
+DATA
 Text HLabel 7375 3800 2    59   Input ~ 0
-A5
+CLK
 Text HLabel 5500 2450 2    59   Input ~ 0
 3.3V

Commit message: feat: add 2 IO, 1 one wire, fan and 3 stepper output. Closes: #20 #11 #9 #4
Parts:
- U4: value HX711HX711 -> HX711
Changed lines of the file:
@@
 P 6725 3500
 F 0 "U4" H 6675 4486 59  0000 C CNN
-F 1 "HX711HX711" H 6675 4381 59  0000 C CNN
+F 1 "HX711" H 6675 4381 59  0000 C CNN
 F 2 "Package_SO:STC_SOP-16_3.9x9.9mm_P1.27mm" H 6725 3500 50  0001 C CNN
 F 3 "" H 6725 3500 50  0001 C CNN
