File: pcb/main/Bertha_main.kicad_pcb (KiCad board)
At the start: 2 copper layers, 100 x 87 mm, 135 parts, among them IC1 SST26VF064B, IC2 DRV8811, J1 RJ12, J10 SJ, J11 SJ, J2 Conn_Coaxial_Power, J3 Conn_02x03_Odd_Even, J4 RJ12, J5 AudioJack3_SwitchTR, J6 SJ, J7 Conn_01x01, J8 Conn_01x01, J9 SJ, Q1 BSP75, Q2 BSP75, Q3 MJH6284, Q4 MMBT4403, U1 DS18B20SMALL, U2 ATMEGA32U4-AU, U3 ACT4088, U4 HX711HX711, X1 MINI-USB-SCHIELD-32005-201, Y1 Crystal

Commit message: fix: update arduino code
Parts:
- D1, D2, D3: value Schottky -> D_Schottky
- IC1: value SST26VF064B -> SST26VF064B-104V_MF
- Q4: value MMBT4403 -> TRANSISTOR_PNPMMBT4403
- SJ1: value JUMPER -> JUMPER-PAD-2-NC_BY_TRACE
Changed lines of the file:
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@@
   (page A4)
   (layers
-    (0 F.Cu signal hide)
-    (31 B.Cu signal hide)
+    (0 F.Cu signal)
+    (31 B.Cu signal)
     (32 B.Adhes user)
     (33 F.Adhes user)
@@
       (effects (font (size 1 1) (thickness 0.15)))
     )
-    (fp_text value Schottky (at 0 -1.397 90) (layer F.Fab)
+    (fp_text value D_Schottky (at 0 -1.397 90) (layer F.Fab)
       (effects (font (size 1 1) (thickness 0.15)))
     )
@@
       (effects (font (size 1 1) (thickness 0.15)))
     )
-    (fp_text value Schottky (at 3.175 -0.254) (layer F.Fab)
+    (fp_text value D_Schottky (at 3.175 -0.254) (layer F.Fab)
       (effects (font (size 1 1) (thickness 0.15)))
     )
@@
       (effects (font (size 1 1) (thickness 0.15)))
     )
-    (fp_text value Schottky (at 3.556 0.127) (layer F.Fab)
+    (fp_text value D_Schottky (at 3.556 0.127) (layer F.Fab)
       (effects (font (size 1 1) (thickness 0.15)))
     )
@@
       (effects (font (size 1 1) (thickness 0.15)))
     )
-    (fp_text value SST26VF064B (at 1.016 0.254) (layer F.Fab)
+    (fp_text value SST26VF064B-104V_MF (at 1.016 0.254) (layer F.Fab)
       (effects (font (size 1 1) (thickness 0.15)))
     )
@@
       (effects (font (size 1 1) (thickness 0.15)))
     )
-    (fp_text value MMBT4403 (at 0.1665 2.4765 -90) (layer F.Fab)
+    (fp_text value TRANSISTOR_PNPMMBT4403 (at 0.1665 2.4765 -90) (layer F.Fab)
       (effects (font (size 1 1) (thickness 0.15)))
     )
@@
       (effects (font (size 1 1) (thickness 0.15)))
     )
-    (fp_text value JUMPER (at -2.4361 2.6035) (layer F.Fab)
+    (fp_text value JUMPER-PAD-2-NC_BY_TRACE (at -2.4361 2.6035) (layer F.Fab)
       (effects (font (size 1 1) (thickness 0.15)))
     )
@@
   (segment (start 140.327639 98.178362) (end 140.327639 98.178361) (width 0.508) (layer F.Cu) (net 33))
   (segment (start 142.748 105.177902) (end 142.769988 105.155914) (width 0.508) (layer B.Cu) (net 33))
-  (via (at 142.748 104.267) (size 1.6) (drill 0.8) (layers F.Cu B.Cu) (net 33))
+  (via (at 142.748 105.029) (size 1.6) (drill 0.8) (layers F.Cu B.Cu) (net 33))
   (segment (start 142.748 105.029) (end 142.748 107.95) (width 0.508) (layer B.Cu) (net 33))
   (via (at 142.748 107.95) (size 1.6) (drill 0.8) (layers F.Cu B.Cu) (net 33))

Commit message: fix(pcb): wrong pad connected in bsp75
Parts:
- Q1, Q2: footprint Package_TO_SOT_SMD:SOT-223-3_TabPin2 -> Bertha_footprints:SOT-223-3_TabPin3
Routing:
- net GND: track 223.7 -> 231.6 mm, vias 38 -> 40
- net Net-(JP4-Pad2): track 11.2 -> 5.00 mm
- net Net-(JP3-Pad2): track 11.0 -> 4.85 mm
Changed lines of the file:
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@@
     (thickness 1.6)
     (drawings 80)
-    (tracks 1031)
+    (tracks 1035)
     (zones 0)
     (modules 135)
@@
   )
   (setup
-    (last_trace_width 0.25)
+    (last_trace_width 2.54)
     (user_trace_width 0.4)
     (user_trace_width 0.508)
@@
     (uvia_drill 0.1)
   )
-  (module Package_TO_SOT_SMD:SOT-223-3_TabPin2 (layer F.Cu)
+  (module Bertha_footprints:SOT-223-3_TabPin3 (layer F.Cu)
     (at 125.584 82.534 270)
     (descr "module CMS SOT223 4 pins")
@@
     (pad 2 smd rect (at -3.15 0 270) (size 2 1.5) (layers F.Cu F.Paste F.Mask)
       (net 87 "Net-(JP4-Pad2)"))
-    (pad 2 smd rect (at 3.15 0 270) (size 2 3.8) (layers F.Cu F.Paste F.Mask)
-      (net 87 "Net-(JP4-Pad2)"))
+    (pad 3 smd rect (at 3.15 0 270) (size 2 3.8) (layers F.Cu F.Paste F.Mask)
+      (net 1 GND))
     (model ${KISYS3DMOD}/Package_TO_SOT_SMD.3dshapes/SOT-223.wrl
       (at (xyz 0 0 0))
@@
     )
   )
-  (module Package_TO_SOT_SMD:SOT-223-3_TabPin2 (layer F.Cu)
+  (module Bertha_footprints:SOT-223-3_TabPin3 (layer F.Cu)
     (at 139.3 82.534 270)
     (descr "module CMS SOT223 4 pins")
@@
     (pad 2 smd rect (at -3.15 0 270) (size 2 1.5) (layers F.Cu F.Paste F.Mask)
       (net 86 "Net-(JP3-Pad2)"))
-    (pad 2 smd rect (at 3.15 0 270) (size 2 3.8) (layers F.Cu F.Paste F.Mask)
-      (net 86 "Net-(JP3-Pad2)"))
+    (pad 3 smd rect (at 3.15 0 270) (size 2 3.8) (layers F.Cu F.Paste F.Mask)
+      (net 1 GND))
     (model ${KISYS3DMOD}/Package_TO_SOT_SMD.3dshapes/SOT-223.wrl
       (at (xyz 0 0 0))
@@
   (segment (start 145.297 116.232798) (end 145.297 117.856) (width 0.508) (layer F.Cu) (net 1))
   (segment (start 147.483001 115.088999) (end 146.440799 115.088999) (width 0.508) (layer F.Cu) (net 1))
+  (via (at 121.92 86.36) (size 2.4) (drill 1.2) (layers F.Cu B.Cu) (net 1))
+  (segment (start 122.596 85.684) (end 121.92 86.36) (width 2.54) (layer F.Cu) (net 1))
+  (segment (start 125.584 85.684) (end 122.596 85.684) (width 2.54) (layer F.Cu) (net 1))
+  (via (at 135.636 86.36) (size 2.4) (drill 1.2) (layers F.Cu B.Cu) (net 1))
+  (segment (start 136.312 85.684) (end 135.636 86.36) (width 2.54) (layer F.Cu) (net 1))
+  (segment (start 139.3 85.684) (end 136.312 85.684) (width 2.54) (layer F.Cu) (net 1))
   (segment (start 143.247 117.156) (end 143.247 117.856) (width 0.508) (layer F.Cu) (net 2))
   (segment (start 146.114001 114.288999) (end 143.247 117.156) (width 0.508) (layer F.Cu) (net 2))
@@
   (segment (start 139.3 77.264959) (end 140.38901 76.175949) (width 2.54) (layer F.Cu) (net 86))
   (segment (start 139.3 79.435) (end 139.3 77.264959) (width 2.54) (layer F.Cu) (net 86))
-  (segment (start 139.3 85.633) (end 139.3 79.435) (width 2.54) (layer F.Cu) (net 86))
   (segment (start 127.05401 76.175949) (end 127.05401 75.041) (width 2.54) (layer F.Cu) (net 87))
   (segment (start 125.584 77.645959) (end 127.05401 76.175949) (width 2.54) (layer F.Cu) (net 87))
   (segment (start 125.584 79.435) (end 125.584 77.645959) (width 2.54) (layer F.Cu) (net 87))
-  (segment (start 125.584 85.633) (end 125.584 79.435) (width 2.54) (layer F.Cu) (net 87))
   (segment (start 105.4615 75.2485) (end 105.9515 74.7585) (width 0.508) (layer F.Cu) (net 88))
   (segment (start 98.730872 81.672628) (end 98.1075 82.296) (width 0.508) (layer F.Cu) (net 88))

Commit message: fix: remove resistor on the GND of onewire
Parts:
- removed R8: 4.7k, Resistor_SMD:R_0805_2012Metric_Pad1.15x1.40mm_HandSolder
Connections:
- J5 pad R: Net-(J5-PadR) -> GND
Routing:
- net GND: track 231.6 -> 222.4 mm
- net Net-(J5-PadR): track 3.76 -> 0.00 mm

Commit message: fix: pcb
Routing:
- net D5: track 53.0 -> 52.5 mm
Changed lines of the file:
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@@
     (thickness 1.6)
     (drawings 82)
-    (tracks 1031)
+    (tracks 1030)
     (zones 0)
     (modules 134)
@@
   (segment (start 129.032 88.138) (end 131.318 90.424) (width 0.508) (layer F.Cu) (net 24))
   (segment (start 129.032 82.04) (end 129.032 88.138) (width 0.508) (layer F.Cu) (net 24))
-  (segment (start 131.318 90.424) (end 130.81 90.424) (width 0.508) (layer F.Cu) (net 24))
   (segment (start 143.256 90.424) (end 131.318 90.424) (width 0.508) (layer F.Cu) (net 24))
   (segment (start 149.983001 104.254001) (end 147.329 101.6) (width 0.508) (layer F.Cu) (net 25))

Commit message: feat(pcb): adding 2 I/O, 1 tmp sensor, 4 stepper
Parts:
- added D18: RED, LED_SMD:LED_0805_2012Metric_Pad1.15x1.40mm_HandSolder, F.Cu at (137.2, 70.5)
- added D19: RED, LED_SMD:LED_0805_2012Metric_Pad1.15x1.40mm_HandSolder, F.Cu at (137.2, 80.6)
- added D20: TX, LED_SMD:LED_0805_2012Metric_Pad1.15x1.40mm_HandSolder, F.Cu at (69.8, 174.0)
- added D21: TX, LED_SMD:LED_0805_2012Metric_Pad1.15x1.40mm_HandSolder, F.Cu at (69.8, 177.0)
- added D22: TX, LED_SMD:LED_0805_2012Metric_Pad1.15x1.40mm_HandSolder, F.Cu at (74.6, 174.0)
- added J12: AudioJack3_SwitchTR, Connector_Audio:Jack_3.5mm_Ledino_KB3SPRS_Horizontal, F.Cu at (120.7, 141.0)
- added JP10: JP4E, Connector_PinHeader_2.54mm:PinHeader_1x04_P2.54mm_Vertical, F.Cu at (161.9, 71.1)
- added JP11: JP4E, Connector_PinHeader_2.54mm:PinHeader_1x04_P2.54mm_Vertical, F.Cu at (161.9, 68.6)
- added JP12: JP4E, Connector_PinHeader_2.54mm:PinHeader_1x04_P2.54mm_Vertical, F.Cu at (161.9, 66.0)
- added JP8: IO3, Connector_PinHeader_2.54mm:PinHeader_1x02_P2.54mm_Vertical, F.Cu at (137.8, 73.0)
- added JP9: IO4, Connector_PinHeader_2.54mm:PinHeader_1x02_P2.54mm_Vertical, F.Cu at (137.8, 83.2)
- added Q5: ZXMS6004, Package_TO_SOT_SMD:SOT-23, F.Cu at (141.6, 76.8)
- added Q6: ZXMS6004, Package_TO_SOT_SMD:SOT-23, F.Cu at (141.6, 87.0)
- added R50: 4.7k, Resistor_SMD:R_0805_2012Metric_Pad1.15x1.40mm_HandSolder, F.Cu at (122.5, 167.6)
- added R51: 1k, Resistor_SMD:R_0805_2012Metric_Pad1.15x1.40mm_HandSolder, F.Cu at (112.1, 167.7)
- added R52: 10k, Resistor_SMD:R_0805_2012Metric_Pad1.15x1.40mm_HandSolder, F.Cu at (141.4, 70.5)
- added R53: 10k, Resistor_SMD:R_0805_2012Metric_Pad1.15x1.40mm_HandSolder, F.Cu at (141.6, 80.6)
- added R54: 1k, Resistor_SMD:R_0805_2012Metric_Pad1.15x1.40mm_HandSolder, F.Cu at (74.6, 177.0)
- added R55: 1k, Resistor_SMD:R_0805_2012Metric_Pad1.15x1.40mm_HandSolder, F.Cu at (79.4, 173.9)
- added R56: 1k, Resistor_SMD:R_0805_2012Metric_Pad1.15x1.40mm_HandSolder, F.Cu at (79.3, 177.0)
- added R8: 100, Resistor_SMD:R_0805_2012Metric_Pad1.15x1.40mm_HandSolder, F.Cu at (107.4, 167.7)
- JP3: value IN -> IO1
- JP4: value OUT -> IO2
- Q1, Q2: value BSP75 -> ZXMS6004; footprint Bertha_footprints:SOT-223-3_TabPin3 -> Package_TO_SOT_SMD:SOT-23
- moved R9 24.8 mm to (142.9, 99.1), turned to 0 degrees
- moved R11 24.1 mm to (142.9, 101.6), turned to 0 degrees
- moved D4 17.1 mm to (146.7, 99.1), turned to 180 degrees
- moved D5 15.9 mm to (146.7, 101.6), turned to 180 degrees
- moved JP3 12.7 mm to (125.1, 73.0)
- moved D8 12.2 mm to (124.5, 70.5)
- moved R17 12.2 mm to (128.9, 70.5)
- moved Q1 11.9 mm to (128.9, 76.8)
- moved D9 9.61 mm to (124.7, 80.5)
- moved R20 9.61 mm to (129.1, 80.5)
- moved JP4 8.15 mm to (124.5, 83.2)
- moved J5 8.13 mm to (134.6, 140.7)
- moved C15 6.48 mm to (178.1, 125.0)
- moved D7 6.48 mm to (180.5, 115.6)
- moved R16 6.48 mm to (184.5, 115.6)
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Connections:
- U2 pad 25: /A6 -> A6
- U2 pad 26: /D12 -> D12
Routing:
- net A6: track 0.00 -> 41.8 mm, vias 0 -> 2
- net D12: track 0.00 -> 30.8 mm, vias 0 -> 2
- net Net-(D1-Pad2): track 42.4 -> 12.9 mm
- net VUSB: track 65.9 -> 42.2 mm
- net 12V: track 336.8 -> 355.0 mm
- net Net-(D20-Pad1): track 22.2 -> 4.50 mm
- net TXLED: track 3.67 -> 21.1 mm, vias 0 -> 2
- net GND: track 222.4 -> 208.2 mm, vias 40 -> 42
- net SCL: track 56.9 -> 42.9 mm
- net Net-(J5-PadT): track 16.4 -> 2.54 mm
- net 3.3V: track 513.3 -> 526.8 mm
- net D10: track 40.0 -> 52.2 mm
- net SDA: track 51.9 -> 41.5 mm
- net /Stepper/AOUT2: track 23.6 -> 33.3 mm
- net D5: track 52.5 -> 42.8 mm
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Other:
- board text added: "Bertha V6.0.0"
- board text added: "I/O"
- board text removed: "Bertha V5.0.0"
- board text removed: "Food"

Commit message: feat: add 2 IO, 1 one wire, fan and 3 stepper output. Closes: #20 #11 #9 #4
Parts:
- added JP13: IO4, Connector_Molex:Molex_KK-254_AE-6410-02A_1x02_P2.54mm_Vertical, F.Cu at (185.4, 109.2)
- added Q7: ZXMS6004, Package_TO_SOT_SMD:SOT-23, F.Cu at (178.4, 109.2)
- D10, D14, D15, D16, D17: value LED -> RED
- D11, D13: value RED -> GREEN
- D18, D19, D8, D9: value RED -> BLUE
- D20, D21, D22, D4: value TX -> YELLOW
- D5: value RX -> YELLOW
- D6: value BLK -> WHITE
- D7: value FLASH -> YELLOW
- JP3, JP4, JP8, JP9: footprint Connector_PinHeader_2.54mm:PinHeader_1x02_P2.54mm_Vertical -> Connector_Molex:Molex_KK-254_AE-6410-02A_1x02_P2.54mm_Vertical
- U1: value DS18B20SMALL -> DS18B20
- U4: value HX711HX711 -> HX711
- moved D20 72.9 mm to (127.6, 129.5), turned to 90 degrees
- moved R54 69.8 mm to (125.7, 129.5), turned to 270 degrees
- moved R56 66.5 mm to (119.4, 123.8), turned to 90 degrees
- moved D22 66.0 mm to (117.5, 123.8), turned to 270 degrees
- moved D21 64.6 mm to (113.7, 129.5), turned to 90 degrees
- moved R55 55.0 mm to (111.8, 129.5), turned to 270 degrees
- moved R8 39.1 mm to (115.6, 129.5), turned to 270 degrees
- moved R51 39.0 mm to (120.0, 129.5), turned to 270 degrees
- moved R50 38.4 mm to (117.5, 129.5), turned to 90 degrees
- moved R5 6.11 mm to (129.5, 129.5), turned to 270 degrees
- moved R13 6.02 mm to (121.3, 123.8), turned to 90 degrees
- moved R6 5.51 mm to (131.4, 129.5), turned to 90 degrees
- moved R7 5.50 mm to (134.0, 129.5), turned to 270 degrees
- moved R12 4.72 mm to (115.6, 123.8), turned to 270 degrees
- moved U1 2.96 mm to (111.8, 123.8), turned to 90 degrees
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Connections:
- R51 pad 2: D7 -> A5
- U2 pad 12: /D11 -> D11
- U2 pad 41: /A5 -> A5
Routing:
- net 12V: track 355.0 -> 409.0 mm
- net 3.3V: track 526.8 -> 569.0 mm, vias 7 -> 8
- net A5: track 0.00 -> 37.9 mm, vias 0 -> 2
- net D6: track 70.5 -> 101.7 mm, vias 6 -> 4
- net Net-(D1-Pad2): track 12.9 -> 40.4 mm
- net VUSB: track 42.2 -> 68.6 mm
- net SCL: track 42.9 -> 64.9 mm, vias 1 -> 2
- net D11: track 0.00 -> 21.7 mm, vias 0 -> 2
- net Net-(D21-Pad1): track 0.00 -> 18.3 mm
- net Net-(J12-PadT): track 0.00 -> 17.9 mm
- net Net-(J5-PadT): track 2.54 -> 17.6 mm
- net Net-(D20-Pad1): track 4.50 -> 18.3 mm
- net SDA: track 41.5 -> 53.7 mm
- net TX: track 18.5 -> 30.2 mm
- net Net-(R12-Pad2): track 5.59 -> 13.3 mm
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Other:
- board text added: "1"
- board text added: "2"
- board text added: "3"
- board text added: "4"
- board text added: "FAN"
- board text added: "⏚"

Commit message: fix: improve label on pcb
Parts:
- Q4: value TRANSISTOR_PNPMMBT4403 -> MMBT4403
- SJ1: value JUMPER-PAD-2-NC_BY_TRACE -> JP
Changed lines of the file:
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@@
   (page A4)
   (layers
-    (0 F.Cu signal)
-    (31 B.Cu signal)
+    (0 F.Cu signal hide)
+    (31 B.Cu signal hide)
     (32 B.Adhes user)
     (33 F.Adhes user)
@@
   )
   (setup
-    (last_trace_width 0.508)
+    (last_trace_width 0.25)
     (user_trace_width 0.4)
     (user_trace_width 0.508)
@@
     (solder_mask_min_width 0.25)
     (aux_axis_origin 0 0)
-    (visible_elements FFFDFF7F)
+    (visible_elements FFFBFF7F)
     (pcbplotparams
       (layerselection 0x010fc_ffffffff)
@@
       (effects (font (size 1 1) (thickness 0.15)))
     )
-    (fp_text value ZXMS6004 (at -2.286 0 180) (layer F.Fab)
+    (fp_text value ZXMS6004 (at 0 -2.54 270) (layer F.Fab)
       (effects (font (size 0.508 0.508) (thickness 0.127)))
     )
@@
       (effects (font (size 1 1) (thickness 0.15)))
     )
-    (fp_text value ZXMS6004 (at -2.286 0 180) (layer F.Fab)
+    (fp_text value ZXMS6004 (at 0 -2.54 270) (layer F.Fab)
       (effects (font (size 0.508 0.508) (thickness 0.127)))
     )
@@
       (effects (font (size 1 1) (thickness 0.15)))
     )
-    (fp_text value ZXMS6004 (at -2.159 0 180) (layer F.Fab)
+    (fp_text value ZXMS6004 (at -0.635 -2.54 270) (layer F.Fab)
       (effects (font (size 0.508 0.508) (thickness 0.127)))
     )
@@
       (effects (font (size 1 1) (thickness 0.15)))
     )
-    (fp_text value ZXMS6004 (at -2.159 0 180) (layer F.Fab)
+    (fp_text value ZXMS6004 (at -0.635 -2.54 270) (layer F.Fab)
       (effects (font (size 0.508 0.508) (thickness 0.127)))
     )
@@
       (effects (font (size 1 1) (thickness 0.15)))
     )
-    (fp_text value SJ (at 0 1.9 270) (layer F.Fab)
+    (fp_text value SJ (at 0 -1.397 270) (layer F.Fab)
       (effects (font (size 1 1) (thickness 0.15)))
     )
@@
       (effects (font (size 1 1) (thickness 0.15)))
     )
-    (fp_text value TRANSISTOR_PNPMMBT4403 (at 0.1665 2.4765 -90) (layer F.Fab)
+    (fp_text value MMBT4403 (at 0.1665 2.4765 -90) (layer F.Fab)
       (effects (font (size 1 1) (thickness 0.15)))
     )
@@
       (effects (font (size 1 1) (thickness 0.15)))
     )
-    (fp_text value JUMPER-PAD-2-NC_BY_TRACE (at -2.4361 2.6035) (layer F.Fab)
+    (fp_text value JP (at -2.4361 0.3175) (layer F.Fab)
       (effects (font (size 1 1) (thickness 0.15)))
     )

Commit message: fix: close https://github.com/Hackuarium/bioreactor/issues/32
Parts:
- Q4: value MMBT4403 -> TRANSISTOR_PNPMMBT4403
- SJ1: value JP -> JUMPER-PAD-2-NC_BY_TRACE
Connections:
- Q1 pad 2: Net-(JP3-Pad2) -> GND
- Q1 pad 3: GND -> Net-(JP3-Pad2)
- Q2 pad 2: Net-(JP4-Pad2) -> GND
- Q2 pad 3: GND -> Net-(JP4-Pad2)
- Q5 pad 2: Net-(JP8-Pad2) -> GND
- Q5 pad 3: GND -> Net-(JP8-Pad2)
- Q6 pad 2: Net-(JP9-Pad2) -> GND
- Q6 pad 3: GND -> Net-(JP9-Pad2)
- Q7 pad 2: Net-(JP13-Pad2) -> GND
- Q7 pad 3: GND -> Net-(JP13-Pad2)
Routing:
- net GND: track 214.3 -> 227.7 mm
- net Net-(JP8-Pad2): track 2.86 -> 6.66 mm
- net Net-(JP9-Pad2): track 2.86 -> 6.66 mm
- net Net-(JP3-Pad2): track 2.86 -> 6.66 mm
- net Net-(JP4-Pad2): track 3.50 -> 6.66 mm
- net Net-(JP13-Pad2): track 3.91 -> 4.86 mm
