File: pcb/main/Bertha_main.kicad_pcb (KiCad board)
At the start: 2 copper layers, 100 x 87 mm, 157 parts, among them IC1 SST26VF064B-104V_MF, IC2 DRV8811, J1 RJ12, J10 SJ, J11 SJ, J12 AudioJack3_SwitchTR, J2 Conn_Coaxial_Power, J3 Conn_02x03_Odd_Even, J4 RJ12, J5 AudioJack3_SwitchTR, J6 SJ, J7 Conn_01x01, J8 Conn_01x01, J9 SJ, Q1 ZXMS6004, Q2 ZXMS6004, Q3 MJH6284, Q4 TRANSISTOR_PNPMMBT4403, Q5 ZXMS6004, Q6 ZXMS6004, Q7 ZXMS6004, U1 DS18B20, U2 ATMEGA32U4-AU, U3 ACT4088, U4 HX711, X1 MINI-USB-SCHIELD-32005-201, Y1 Crystal

Commit message: fix: suppress leds for onewire
Parts:
- removed D20, D21, D22: YELLOW, LED_SMD:LED_0805_2012Metric_Pad1.15x1.40mm_HandSolder
- removed R54, R55, R56: 1k, Resistor_SMD:R_0805_2012Metric_Pad1.15x1.40mm_HandSolder
- moved R13 3.81 mm to (117.5, 123.8)
Routing:
- net 3.3V: track 569.0 -> 554.5 mm
- net Net-(R12-Pad2): track 13.3 -> 7.99 mm
- net A2: track 31.9 -> 35.8 mm
- net Net-(D22-Pad2): track 1.91 -> 0.00 mm
- net Net-(D21-Pad2): track 1.91 -> 0.00 mm
- net Net-(D20-Pad2): track 1.91 -> 0.00 mm
- net Net-(J5-PadS): track 18.3 -> 16.4 mm
- net Net-(J12-PadS): track 18.3 -> 16.4 mm

Commit message: Changed MJH6284 darlington transistor for two PB80N03S4L03 MOSFETs
Parts:
- added C34: 4n, Capacitor_SMD:C_0805_2012Metric_Pad1.15x1.40mm_HandSolder, F.Cu at (37.4, 136.5)
- added C35: 4n, Capacitor_SMD:C_0805_2012Metric_Pad1.15x1.40mm_HandSolder, F.Cu at (42.2, 136.5)
- added Q8: IPB80N03S4L-03, Package_TO_SOT_SMD:TO-263-2, F.Cu at (40.6, 114.3)
- added R54: 330, Resistor_SMD:R_0805_2012Metric_Pad1.15x1.40mm_HandSolder, F.Cu at (93.7, 127.8)
- Q3: value MJH6284 -> IPB80N03S4L-03; footprint Package_TO_SOT_THT:TO-247-3_Vertical -> Package_TO_SOT_SMD:TO-263-2
- R19: value 100 -> 330
- moved Q3 33.3 mm to (58.4, 116.4), turned to 90 degrees
Routing:
- net Net-(J8-Pad1): track 13.0 -> 0.00 mm
- net Net-(C34-Pad1): track 8.99 -> 0.00 mm

Commit message: Update PCB wih new PID control
Parts:
- removed C35: 4n, Capacitor_SMD:C_0805_2012Metric_Pad1.15x1.40mm_HandSolder
- removed Q8: IPB80N03S4L-03, Package_TO_SOT_SMD:TO-263-2
- removed R54: 330, Resistor_SMD:R_0805_2012Metric_Pad1.15x1.40mm_HandSolder
- moved C34 55.2 mm to (92.5, 132.1)
- moved Q3 38.5 mm to (96.5, 121.9)
- moved D10 12.1 mm to (102.9, 128.0), turned to 270 degrees
- moved R19 6.04 mm to (91.4, 135.9), turned to 270 degrees
- moved R21 2.96 mm to (94.6, 135.9), turned to 90 degrees
Routing:
- net D6: track 101.7 -> 87.1 mm
- net GND: track 227.7 -> 241.2 mm
- net Net-(J8-Pad1): track 0.00 -> 9.66 mm, vias 0 -> 67
- net Net-(D10-Pad2): track 2.79 -> 11.2 mm
- net Net-(C34-Pad1): track 0.00 -> 8.22 mm
- net A5: track 37.9 -> 36.0 mm
- added copper zone on F.Cu, net GND
- added copper zone on B.Cu, net Net-(J8-Pad1)
- added copper zone on F.Cu, net Net-(J8-Pad1)

Commit message: Created ERROR LED & FAN LED
Parts:
- added C35: 100n, Capacitor_SMD:C_0805_2012Metric_Pad1.15x1.40mm_HandSolder, F.Cu at (175.0, 109.2)
- added D20: RED, LED_SMD:LED_0805_2012Metric_Pad1.15x1.40mm_HandSolder, F.Cu at (127.9, 93.3)
- added D21: RED, LED_SMD:LED_0805_2012Metric_Pad1.15x1.40mm_HandSolder, F.Cu at (179.7, 110.1)
- added JP14: IO4, Connector_Molex:Molex_KK-254_AE-6410-02A_1x02_P2.54mm_Vertical, F.Cu at (135.9, 93.3)
- added R54: 10k, Resistor_SMD:R_0805_2012Metric_Pad1.15x1.40mm_HandSolder, F.Cu at (131.8, 93.3)
- added R55: 10k, Resistor_SMD:R_0805_2012Metric_Pad1.15x1.40mm_HandSolder, F.Cu at (175.0, 111.1)
- C34: value 4n -> 100n
- R19: value 330 -> 100
- moved Q7 4.49 mm to (175.3, 106.0)
Connections:
- U2 pad 40: /A4 -> A4
Routing:
- net A4: track 0.00 -> 30.1 mm, vias 0 -> 1
- net 3.3V: track 554.5 -> 563.0 mm
- net D11: track 21.7 -> 30.1 mm
- net Net-(JP13-Pad2): track 4.86 -> 10.5 mm
- net GND: track 241.2 -> 235.8 mm, vias 44 -> 43
- net D12: track 30.1 -> 34.8 mm
- net Net-(D21-Pad2): track 0.00 -> 3.67 mm
- net TXLED: track 21.1 -> 24.4 mm
- net A6: track 42.4 -> 45.1 mm
- net A2: track 35.8 -> 37.9 mm
- net Net-(D20-Pad2): track 0.00 -> 1.91 mm
- net RXLED: track 19.3 -> 20.4 mm
- net D10: track 53.3 -> 52.7 mm, vias 0 -> 2
- net D5: track 42.1 -> 42.4 mm, vias 0 -> 2
Other:
- board text added: "3V3 BUCK"
- board text added: "ERROR"
- board text removed: "3.3V BUCK"

Commit message: Deleted unnecessary resistor and add capacitors to VMA & VMB DRV8811 (issue #28)
Parts:
- removed R35, R37, R38: 10k, Resistor_SMD:R_0805_2012Metric_Pad1.15x1.40mm_HandSolder
- added C36: 100n, Capacitor_SMD:C_0805_2012Metric_Pad1.15x1.40mm_HandSolder, F.Cu at (173.6, 83.8)
- added C37: 100n, Capacitor_SMD:C_0805_2012Metric_Pad1.15x1.40mm_HandSolder, F.Cu at (159.6, 83.8)
- moved R49 1.69 mm to (170.8, 80.9)
- moved C25 1.29 mm to (150.5, 81.3)
- moved R34 0.89 mm to (153.0, 73.9)
- moved C28 0.63 mm to (178.1, 88.6)
- moved R43 0.22 mm to (174.6, 88.6)
- turned C23 to 90 degrees
Connections:
- IC2 pad 26: Net-(IC2-Pad26) -> GND
- IC2 pad 27: Net-(IC2-Pad27) -> 3.3V
Routing:
- net GND: track 235.8 -> 212.4 mm
- net 3.3V: track 563.0 -> 552.4 mm, vias 8 -> 7
- net Net-(IC2-Pad27): track 3.87 -> 0.00 mm
- net Net-(IC2-Pad17): track 3.65 -> 0.00 mm
- net Net-(IC2-Pad26): track 3.28 -> 0.00 mm
- net A6: track 45.1 -> 43.1 mm
- net 12V: track 409.0 -> 407.6 mm
- net D12: track 34.8 -> 33.7 mm
- net Net-(C23-Pad2): track 9.57 -> 10.4 mm
- net /Stepper/AOUT2: track 33.3 -> 34.1 mm
- net Net-(IC2-Pad16): track 4.22 -> 3.67 mm

Commit message: New place for ERROR and add transistor for LED-strip (issue #37)
Parts:
- added C38: 100n, Capacitor_SMD:C_0805_2012Metric_Pad1.15x1.40mm_HandSolder, F.Cu at (142.6, 122.6)
- added Q8: ZXMS6004, Package_TO_SOT_SMD:SOT-23, F.Cu at (142.9, 119.7)
- moved D20 35.0 mm to (142.6, 125.1), turned to 180 degrees
- moved JP14 32.3 mm to (146.7, 123.8)
- moved R54 28.0 mm to (139.6, 120.3), turned to 270 degrees
- moved C7 3.83 mm to (145.3, 116.5), turned to 90 degrees
- moved C11 3.36 mm to (141.6, 115.8), turned to 270 degrees
- moved R2 1.91 mm to (142.2, 133.1)
- moved R6 1.91 mm to (129.5, 129.5)
- moved R7 1.91 mm to (132.1, 129.5)
- moved R5 1.90 mm to (127.6, 129.5)
Connections:
- JP14 pad 1: A4 -> 12V
- JP14 pad 2: GND -> Net-(JP14-Pad2)
Routing:
- net 3.3V: track 552.4 -> 542.0 mm
- net Net-(JP14-Pad2): track 0.00 -> 9.95 mm
- net 12V: track 407.6 -> 415.2 mm
- net D6: track 87.5 -> 81.6 mm, vias 4 -> 2
- net Net-(D1-Pad2): track 40.4 -> 44.2 mm
- net Net-(D20-Pad2): track 1.91 -> 5.40 mm
- net D7: track 23.1 -> 26.2 mm
- net VUSB: track 68.6 -> 71.7 mm
- net A4: track 30.1 -> 27.8 mm, vias 1 -> 2
- net A2: track 37.9 -> 35.7 mm
- net A5: track 36.0 -> 34.5 mm
- net SDA: track 53.7 -> 52.9 mm
- net GND: track 212.4 -> 211.7 mm, vias 43 -> 48
- net Net-(J5-PadS): track 16.4 -> 15.8 mm
Other:
- board text added: "Bertha V6.0.1"
- board text removed: "Bertha V6.0.0"

Commit message: Solved debug error for PID
Parts:
- moved D10 0.63 mm to (102.9, 128.7)
- moved Q8 0.43 mm to (142.4, 119.7)
- moved C37 0.19 mm to (159.5, 83.9)
Routing:
- net GND: track 211.7 -> 217.0 mm
- net A4: track 27.8 -> 25.0 mm
- net 3.3V: track 542.0 -> 544.0 mm
- net 12V: track 415.2 -> 416.3 mm
- net D6: track 81.6 -> 82.6 mm
- net Net-(JP14-Pad2): track 9.95 -> 9.26 mm
- net Net-(J8-Pad1): vias 67 -> 0

Commit message: chore: move values labels
Parts:
- D1, D2, D3: value D_Schottky -> Schottky
- IC1: value SST26VF064B-104V_MF -> SST26VF064B
- J2: value Conn_Coaxial_Power -> Barel
- J3: value Conn_02x03_Odd_Even -> 02x03
- Q4: value TRANSISTOR_PNPMMBT4403 -> MMBT4403
- SJ1: value JUMPER-PAD-2-NC_BY_TRACE -> JP
Other:
- board text added: "Bertha V6.0.2"
- board text removed: "Bertha V6.0.1"
