File: pcb/main/Bertha_main.kicad_pcb (KiCad board)
At the start: 2 copper layers, 100 x 87 mm, 159 parts, among them IC1 SST26VF064B, IC2 DRV8811, J1 RJ12, J10 SJ, J11 SJ, J12 AudioJack3_SwitchTR, J2 Barel, J3 02x03, J4 RJ12, J5 AudioJack3_SwitchTR, J6 SJ, J7 Conn_01x01, J8 Conn_01x01, J9 SJ, Q1 ZXMS6004, Q2 ZXMS6004, Q3 IPB80N03S4L-03, Q4 MMBT4403, Q5 ZXMS6004, Q6 ZXMS6004, Q7 ZXMS6004, Q8 ZXMS6004, U1 DS18B20, U2 ATMEGA32U4-AU, U3 ACT4088, U4 HX711, X1 MINI-USB-SCHIELD-32005-201, Y1 Crystal

Commit message: chore: format update
Other:
- net class Default removed
- net class Safe removed
- board text added: "Bertha V6.1.1"
- board text removed: "1"
- board text removed: "Bertha V6.0.2"
- board text removed: "Flash"
- board text removed: "I/O"
- board text removed: "Load Cell"
- board text removed: "PID"

Commit message: Update 2: Fields for BOM with PCBA manufacturer
Parts:
- C1, C17, C21, C3, C4: value 10uF -> 10u
- C10, C9: value 22pF -> 22p; footprint Capacitor_SMD:C_1206_3216Metric_Pad1.42x1.75mm_HandSolder -> Capacitor_SMD:C_0805_2012Metric_Pad1.18x1.45mm_HandSolder
- C11, C15, C16, C18, C19, C2, C20, C24, C27, C28, C29, C32, C33, C5, C6, C7, C8: value 100nF -> 100n
- C12: value 22nF -> 22n
- C13: value 10µF -> 10u
- C14: value 22µF -> 22u
- C22, C23, C26: value 220nF -> 220n
- C25: value 100uF 50V -> 100u
- C30, C31: value 1nF -> 1n
- D1, D2, D3: value Schottky -> MBR0520LT1G
- D12: footprint Diode_SMD:D_SOD-123 -> Diode_SMD:D_SMA
- IC1: value SST26VF064B -> SST26VF064B-104V
- J2: value Barel -> Conn_Coaxial_Power
- J3: value 02x03 -> Conn_02x03_Odd_Even
- L1: value 4.7µH -> 4.7u
- Q4: value MMBT4403 -> TRANSISTOR_PNPMMBT4403
- R43, R44: value 0.1R 1W -> 0.1
- SJ1: value JP -> JUMPER-PAD-2-NC_BY_TRACE
- moved C12 0.44 mm to (129.8, 103.8)
Connections:
- Q3 pad 10: Net-(J8-Pad1) -> (no net)
- Q3 pad 11: Net-(J8-Pad1) -> (no net)
- Q3 pad 12: Net-(J8-Pad1) -> (no net)
- Q3 pad 13: Net-(J8-Pad1) -> (no net)
- Q3 pad 14: Net-(J8-Pad1) -> (no net)
- Q3 pad 15: Net-(J8-Pad1) -> (no net)
- Q3 pad 4: Net-(J8-Pad1) -> (no net)
- Q3 pad 5: Net-(J8-Pad1) -> (no net)
- Q3 pad 6: Net-(J8-Pad1) -> (no net)
- Q3 pad 7: Net-(J8-Pad1) -> (no net)
- Q3 pad 8: Net-(J8-Pad1) -> (no net)
- Q3 pad 9: Net-(J8-Pad1) -> (no net)
Routing:
- net 3.3V: track 544.0 -> 544.9 mm
- net GND: vias 48 -> 47

Commit message: Update 5 - BOM for PCBA. Check 1 issue #46
Parts:
- D12: value B240A -> MBR0520LT1G; footprint Diode_SMD:D_SMA -> Diode_SMD:D_SOD-123
- D6: value WHITE -> GREEN
- R47: value Rlim -> 180
- moved D12 0.13 mm to (130.2, 100.8)

Commit message: docs(BOM): iBOM.html updated
Routing:
- net A6: track 43.1 -> 41.8 mm
