File: pcb/main/Bertha_main.sch (KiCad schematic (older format))
At the start: 79 parts, among them J1 RJ12, J12 AudioJack3_SwitchTR, J2 Conn_Coaxial_Power, J3 Conn_02x03_Odd_Even, J4 RJ12, J5 AudioJack3_SwitchTR, J6 SJ, J7 Conn_01x01, J8 Conn_01x01, Q1 ZXMS6004, Q2 ZXMS6004, Q3 IPB80N03S4L-03, Q5 ZXMS6004, Q6 ZXMS6004, Q7 ZXMS6004, U1 DS18B20, U2 ATMEGA32U4-AU, X1 MINI-USB-SCHIELD-32005-201, Y1 Crystal

Commit message: Created ERROR LED & FAN LED
Parts:
- added C35: 100n, Capacitor_SMD:C_0805_2012Metric_Pad1.15x1.40mm_HandSolder, symbol Device:C
- added D20, D21: RED, LED_SMD:LED_0805_2012Metric_Pad1.15x1.40mm_HandSolder, symbol Device:LED
- added JP14: IO4, Connector_Molex:Molex_KK-254_AE-6410-02A_1x02_P2.54mm_Vertical, symbol Bertha_main-eagle-import:JP1E
- added R54, R55: 10k, Resistor_SMD:R_0805_2012Metric_Pad1.15x1.40mm_HandSolder, symbol Device:R
- C34: value 4n -> 100n
- R19: value 330 -> 100
Connections:
- net A4: now also JP14.1, R54.1
- net D11: now also C35.1, R55.1
- net at Q7.2 (S): now also C35.2, D21.1 (K)
- new net: D21.2 (A), R55.2
- new net: D20.1 (K), JP14.2
- new net: D20.2 (A), R54.2
- no-connect marks 9 -> 8
Other:
- note added: "ERROR"
- moved on the sheet: JP13, Q7
Changed lines of the file:
@@
 AR Path="/5E2163A8" Ref="R19"  Part="1"
 F 0 "R19" V 8175 6975 50  0000 L CNN
-F 1 "330" V 8250 7025 50  0000 L CNN
+F 1 "100" V 8250 7025 50  0000 L CNN
 F 2 "Resistor_SMD:R_0805_2012Metric_Pad1.15x1.40mm_HandSolder" V 8180 7100 50  0001 C CNN
 F 3 "~" H 8250 7100 50  0001 C CNN
@@
 Wire Wire Line
 	4275 4550 4425 4550
-NoConn ~ 4425 4250
 NoConn ~ 4425 4350
 Wire Wire Line
@@
 Wire Wire Line
 	4275 6650 4425 6650
-Text GLabel 6325 8825 0    55   Input ~ 0
+Text GLabel 6800 8700 0    55   Input ~ 0
 12V
 Wire Wire Line
-	6200 8925 6400 8925
-Wire Wire Line
-	6200 9525 6200 9425
+	6675 8800 6875 8800
 $Comp
 L Bertha_main-eagle-import:JP1E JP?
 U 1 1 5F60B538
-P 6500 8825
+P 6975 8700
 AR Path="/5E0D793B/5F60B538" Ref="JP?"  Part="1"
 AR Path="/5F60B538" Ref="JP13"  Part="1"
-F 0 "JP13" V 6575 8925 59  0000 L CNN
-F 1 "IO4" V 6450 8950 59  0000 L CNN
-F 2 "Connector_Molex:Molex_KK-254_AE-6410-02A_1x02_P2.54mm_Vertical" H 6500 8825 50  0001 C CNN
-F 3 "" H 6500 8825 50  0001 C CNN
-	1    6500 8825
+F 0 "JP13" V 7050 8800 59  0000 L CNN
+F 1 "IO4" V 6925 8825 59  0000 L CNN
+F 2 "Connector_Molex:Molex_KK-254_AE-6410-02A_1x02_P2.54mm_Vertical" H 6975 8700 50  0001 C CNN
+F 3 "" H 6975 8700 50  0001 C CNN
+	1    6975 8700
 	0    1    1    0
 $EndComp
 Wire Wire Line
-	6325 8825 6400 8825
-Wire Wire Line
-	6200 9025 6200 8925
+	6800 8700 6875 8700
+Wire Wire Line
+	6675 8900 6675 8800
 $Comp
 L Bertha_main-eagle-import:GND #U0103
 U 1 1 5F60B547
-P 6200 9625
-F 0 "#U0103" H 6250 9675 50  0001 C CNN
-F 1 "GND" H 6303 9663 42  0000 L CNN
-F 2 "" H 6200 9625 50  0001 C CNN
-F 3 "" H 6200 9625 50  0001 C CNN
-	1    6200 9625
-	1    0    0    -1
-$EndComp
-Wire Wire Line
-	5800 9225 6000 9225
+P 6675 9625
+F 0 "#U0103" H 6725 9675 50  0001 C CNN
+F 1 "GND" H 6778 9663 42  0000 L CNN
+F 2 "" H 6675 9625 50  0001 C CNN
+F 3 "" H 6675 9625 50  0001 C CNN
+	1    6675 9625
+	1    0    0    -1
+$EndComp
+Wire Wire Line
+	5675 9100 5950 9100
 $Comp
 L ZXMS6004:ZXMS6004 Q7
 U 1 1 5F60B54F
-P 6200 9225
-F 0 "Q7" H 6306 9271 50  0000 L CNN
-F 1 "ZXMS6004" H 6306 9180 50  0000 L CNN
-F 2 "Package_TO_SOT_SMD:SOT-23" H 6300 9150 50  0001 L CIN
-F 3 "https://www.diodes.com/assets/Datasheets/ZXMS6004FF.pdf" H 6300 9300 50  0001 L CNN
-	1    6200 9225
+P 6675 9100
+F 0 "Q7" H 6781 9146 50  0000 L CNN
+F 1 "ZXMS6004" H 6781 9055 50  0000 L CNN
+F 2 "Package_TO_SOT_SMD:SOT-23" H 6775 9025 50  0001 L CIN
+F 3 "https://www.diodes.com/assets/Datasheets/ZXMS6004FF.pdf" H 6775 9175 50  0001 L CNN
+	1    6675 9100
 	1    0    0    -1
 $EndComp
@@
 	5400 8375 5400 9750
 Wire Notes Line
-	5400 9750 6925 9750
-Wire Notes Line
-	6925 9750 6925 8375
-Wire Notes Line
-	6925 8375 5400 8375
+	7375 9750 7375 8375
 Text GLabel 4425 5450 2    55   Input ~ 0
 D11
 Wire Wire Line
 	4275 5450 4425 5450
-Text GLabel 5800 9225 0    55   Input ~ 0
+Text GLabel 5675 9100 0    55   Input ~ 0
 D11
 Wire Wire Line
@@
 AR Path="/5F59928D" Ref="C34"  Part="1"
 F 0 "C34" H 8250 7275 50  0000 L CNN
-F 1 "4n" H 8300 7200 50  0000 L CNN
+F 1 "100n" H 8300 7200 50  0000 L CNN
 F 2 "Capacitor_SMD:C_0805_2012Metric_Pad1.15x1.40mm_HandSolder" H 8538 7150 50  0001 C CNN
 F 3 "~" H 8500 7300 50  0001 C CNN
@@
 Wire Notes Line
 	7575 6025 10625 6025
+$Comp
+L Device:R R?
+U 1 1 5F4B01F7
+P 5950 9300
+AR Path="/5E0D7B15/5F4B01F7" Ref="R?"  Part="1"
+AR Path="/5F4B01F7" Ref="R55"  Part="1"
+F 0 "R55" V 5875 9175 50  0000 L CNN
+F 1 "10k" V 5950 9225 50  0000 L CNN
+F 2 "Resistor_SMD:R_0805_2012Metric_Pad1.15x1.40mm_HandSolder" V 5880 9300 50  0001 C CNN
+F 3 "~" H 5950 9300 50  0001 C CNN
+	1    5950 9300
+	1    0    0    -1
+$EndComp
+$Comp
+L Device:C C?
+U 1 1 5F4B2617
+P 6400 9300
+AR Path="/5E02557B/5F4B2617" Ref="C?"  Part="1"
+AR Path="/5F4B2617" Ref="C35"  Part="1"
+F 0 "C35" H 6150 9275 50  0000 L CNN
+F 1 "100n" H 6200 9200 50  0000 L CNN
+F 2 "Capacitor_SMD:C_0805_2012Metric_Pad1.15x1.40mm_HandSolder" H 6438 9150 50  0001 C CNN
+F 3 "~" H 6400 9300 50  0001 C CNN
+	1    6400 9300
+	-1   0    0    -1
+$EndComp
+Wire Wire Line
+	6675 9300 6675 9500
+Wire Wire Line
+	6400 9450 6400 9500
+Wire Wire Line
+	6400 9500 6675 9500
+Connection ~ 6675 9500
+Wire Wire Line
+	6675 9500 6675 9525
+Connection ~ 6400 9500
+Wire Wire Line
+	6325 9500 6400 9500
+$Comp
+L Device:LED D?
+U 1 1 5F4B1306
+P 6175 9500
+AR Path="/5E0005EE/5F4B1306" Ref="D?"  Part="1"
+AR Path="/5F4B1306" Ref="D21"  Part="1"
+F 0 "D21" H 6175 9425 50  0000 C CNN
+F 1 "RED" H 6175 9600 50  0000 C CNN
+F 2 "LED_SMD:LED_0805_2012Metric_Pad1.15x1.40mm_HandSolder" H 6175 9500 50  0001 C CNN
+F 3 "~" H 6175 9500 50  0001 C CNN
+	1    6175 9500
+	-1   0    0    -1
+$EndComp
+Wire Wire Line
+	6400 9150 6400 9100
+Wire Wire Line
+	6400 9100 6475 9100
+Wire Wire Line
+	6025 9500 5950 9500
+Wire Wire Line
+	5950 9500 5950 9450
+Wire Wire Line
+	5950 9150 5950 9100
+Connection ~ 5950 9100
+Wire Wire Line
+	5950 9100 6400 9100
+Connection ~ 6400 9100
+Wire Notes Line
+	5400 9750 7375 9750
+Wire Notes Line
+	5400 8375 7375 8375
+Text Notes 975  8000 0    157  ~ 0
+ERROR
+$Comp
+L Bertha_main-eagle-import:JP1E JP?
+U 1 1 5F6B070F
+P 2075 8200
+AR Path="/5E0D793B/5F6B070F" Ref="JP?"  Part="1"
+AR Path="/5F6B070F" Ref="JP14"  Part="1"
+F 0 "JP14" V 2150 8300 59  0000 L CNN
+F 1 "IO4" V 2025 8325 59  0000 L CNN
+F 2 "Connector_Molex:Molex_KK-254_AE-6410-02A_1x02_P2.54mm_Vertical" H 2075 8200 50  0001 C CNN
+F 3 "" H 2075 8200 50  0001 C CNN
+	1    2075 8200
+	0    1    1    0
+$EndComp
+$Comp
+L Device:LED D?
+U 1 1 5F6B0F69
+P 1575 8600
+AR Path="/5E0005EE/5F6B0F69" Ref="D?"  Part="1"
+AR Path="/5F6B0F69" Ref="D20"  Part="1"
+F 0 "D20" H 1575 8525 50  0000 C CNN
+F 1 "RED" H 1575 8700 50  0000 C CNN
+F 2 "LED_SMD:LED_0805_2012Metric_Pad1.15x1.40mm_HandSolder" H 1575 8600 50  0001 C CNN
+F 3 "~" H 1575 8600 50  0001 C CNN
+	1    1575 8600
+	-1   0    0    -1
+$EndComp
+$Comp
+L Device:R R?
+U 1 1 5F6B1D75
+P 1350 8400
+AR Path="/5E0D7B15/5F6B1D75" Ref="R?"  Part="1"
+AR Path="/5F6B1D75" Ref="R54"  Part="1"
+F 0 "R54" V 1275 8275 50  0000 L CNN
+F 1 "10k" V 1350 8325 50  0000 L CNN
+F 2 "Resistor_SMD:R_0805_2012Metric_Pad1.15x1.40mm_HandSolder" V 1280 8400 50  0001 C CNN
+F 3 "~" H 1350 8400 50  0001 C CNN
+	1    1350 8400
+	1    0    0    -1
+$EndComp
+Text GLabel 4425 4250 2    50   Input ~ 0
+A4
+Text GLabel 1175 8200 0    50   Input ~ 0
+A4
+Wire Wire Line
+	1975 8200 1350 8200
+Wire Wire Line
+	1350 8250 1350 8200
+Connection ~ 1350 8200
+Wire Wire Line
+	1350 8200 1175 8200
+Wire Wire Line
+	1425 8600 1350 8600
+Wire Wire Line
+	1350 8600 1350 8550
+$Comp
+L Bertha_main-eagle-import:GND #0102
+U 1 1 5F75493A
+P 1925 8750
+F 0 "#0102" H 1975 8800 50  0001 C CNN
+F 1 "GND" H 2028 8788 42  0000 L CNN
+F 2 "" H 1925 8750 50  0001 C CNN
+F 3 "" H 1925 8750 50  0001 C CNN
+	1    1925 8750
+	1    0    0    -1
+$EndComp
+Wire Wire Line
+	1975 8300 1925 8300
+Wire Wire Line
+	1925 8300 1925 8600
+Wire Wire Line
+	1725 8600 1925 8600
+Connection ~ 1925 8600
+Wire Wire Line
+	1925 8600 1925 8650
+Wire Notes Line
+	875  7750 2475 7750
+Wire Notes Line
+	2475 7750 2475 8850
+Wire Notes Line
+	2475 8850 875  8850
+Wire Notes Line
+	875  8850 875  7750
 $EndSCHEMATC

Commit message: New place for ERROR and add transistor for LED-strip (issue #37)
Parts:
- added C38: 100n, Capacitor_SMD:C_0805_2012Metric_Pad1.15x1.40mm_HandSolder, symbol Device:C
- added Q8: ZXMS6004, Package_TO_SOT_SMD:SOT-23, symbol ZXMS6004:ZXMS6004
Connections:
- net 12V: now also JP14.1
- net A4: now also C38.1, Q8.1 (G); no longer JP14.1
- net at D20.1 (K): now also C38.2, Q8.2 (S); no longer JP14.2
- new net: JP14.2, Q8.3 (D)
Other:
- moved on the sheet: D20, JP14, R54
Changed lines of the file:
@@
 L Bertha_main-eagle-import:JP1E JP?
 U 1 1 5F6B070F
-P 2075 8200
+P 2100 8125
 AR Path="/5E0D793B/5F6B070F" Ref="JP?"  Part="1"
 AR Path="/5F6B070F" Ref="JP14"  Part="1"
-F 0 "JP14" V 2150 8300 59  0000 L CNN
-F 1 "IO4" V 2025 8325 59  0000 L CNN
-F 2 "Connector_Molex:Molex_KK-254_AE-6410-02A_1x02_P2.54mm_Vertical" H 2075 8200 50  0001 C CNN
-F 3 "" H 2075 8200 50  0001 C CNN
-	1    2075 8200
+F 0 "JP14" V 2175 8225 59  0000 L CNN
+F 1 "IO4" V 2050 8250 59  0000 L CNN
+F 2 "Connector_Molex:Molex_KK-254_AE-6410-02A_1x02_P2.54mm_Vertical" H 2100 8125 50  0001 C CNN
+F 3 "" H 2100 8125 50  0001 C CNN
+	1    2100 8125
 	0    1    1    0
 $EndComp
@@
 L Device:LED D?
 U 1 1 5F6B0F69
-P 1575 8600
+P 1450 8925
 AR Path="/5E0005EE/5F6B0F69" Ref="D?"  Part="1"
 AR Path="/5F6B0F69" Ref="D20"  Part="1"
-F 0 "D20" H 1575 8525 50  0000 C CNN
-F 1 "RED" H 1575 8700 50  0000 C CNN
-F 2 "LED_SMD:LED_0805_2012Metric_Pad1.15x1.40mm_HandSolder" H 1575 8600 50  0001 C CNN
-F 3 "~" H 1575 8600 50  0001 C CNN
-	1    1575 8600
+F 0 "D20" H 1450 8850 50  0000 C CNN
+F 1 "RED" H 1450 9025 50  0000 C CNN
+F 2 "LED_SMD:LED_0805_2012Metric_Pad1.15x1.40mm_HandSolder" H 1450 8925 50  0001 C CNN
+F 3 "~" H 1450 8925 50  0001 C CNN
+	1    1450 8925
 	-1   0    0    -1
 $EndComp
@@
 L Device:R R?
 U 1 1 5F6B1D75
-P 1350 8400
+P 1225 8725
 AR Path="/5E0D7B15/5F6B1D75" Ref="R?"  Part="1"
 AR Path="/5F6B1D75" Ref="R54"  Part="1"
-F 0 "R54" V 1275 8275 50  0000 L CNN
-F 1 "10k" V 1350 8325 50  0000 L CNN
-F 2 "Resistor_SMD:R_0805_2012Metric_Pad1.15x1.40mm_HandSolder" V 1280 8400 50  0001 C CNN
-F 3 "~" H 1350 8400 50  0001 C CNN
-	1    1350 8400
+F 0 "R54" V 1150 8600 50  0000 L CNN
+F 1 "10k" V 1225 8650 50  0000 L CNN
+F 2 "Resistor_SMD:R_0805_2012Metric_Pad1.15x1.40mm_HandSolder" V 1155 8725 50  0001 C CNN
+F 3 "~" H 1225 8725 50  0001 C CNN
+	1    1225 8725
 	1    0    0    -1
 $EndComp
 Text GLabel 4425 4250 2    50   Input ~ 0
 A4
-Text GLabel 1175 8200 0    50   Input ~ 0
+Text GLabel 1050 8525 0    50   Input ~ 0
 A4
 Wire Wire Line
-	1975 8200 1350 8200
+	1225 8575 1225 8525
 Wire Wire Line
-	1350 8250 1350 8200
-Connection ~ 1350 8200
+	1225 8525 1050 8525
 Wire Wire Line
-	1350 8200 1175 8200
+	1300 8925 1225 8925
 Wire Wire Line
-	1425 8600 1350 8600
-Wire Wire Line
-	1350 8600 1350 8550
+	1225 8925 1225 8875
 $Comp
 L Bertha_main-eagle-import:GND #0102
 U 1 1 5F75493A
-P 1925 8750
-F 0 "#0102" H 1975 8800 50  0001 C CNN
-F 1 "GND" H 2028 8788 42  0000 L CNN
-F 2 "" H 1925 8750 50  0001 C CNN
-F 3 "" H 1925 8750 50  0001 C CNN
-	1    1925 8750
+P 1950 9075
+F 0 "#0102" H 2000 9125 50  0001 C CNN
+F 1 "GND" H 2053 9113 42  0000 L CNN
+F 2 "" H 1950 9075 50  0001 C CNN
+F 3 "" H 1950 9075 50  0001 C CNN
+	1    1950 9075
 	1    0    0    -1
 $EndComp
 Wire Wire Line
-	1975 8300 1925 8300
+	2000 8225 1950 8225
 Wire Wire Line
-	1925 8300 1925 8600
-Wire Wire Line
-	1725 8600 1925 8600
-Connection ~ 1925 8600
-Wire Wire Line
-	1925 8600 1925 8650
+	1600 8925 1675 8925
 Wire Notes Line
 	875  7750 2475 7750
 Wire Notes Line
-	2475 7750 2475 8850
+	2475 9150 875  9150
+$Comp
+L ZXMS6004:ZXMS6004 Q8
+U 1 1 5F4A21DB
+P 1950 8525
+F 0 "Q8" H 2056 8571 50  0000 L CNN
+F 1 "ZXMS6004" H 2056 8480 50  0000 L CNN
+F 2 "Package_TO_SOT_SMD:SOT-23" H 2050 8450 50  0001 L CIN
+F 3 "https://www.diodes.com/assets/Datasheets/ZXMS6004FF.pdf" H 2050 8600 50  0001 L CNN
+	1    1950 8525
+	1    0    0    -1
+$EndComp
+$Comp
+L Device:C C?
+U 1 1 5F4A3E1A
+P 1675 8725
+AR Path="/5E02557B/5F4A3E1A" Ref="C?"  Part="1"
+AR Path="/5F4A3E1A" Ref="C38"  Part="1"
+F 0 "C38" H 1425 8700 50  0000 L CNN
+F 1 "100n" H 1475 8625 50  0000 L CNN
+F 2 "Capacitor_SMD:C_0805_2012Metric_Pad1.15x1.40mm_HandSolder" H 1713 8575 50  0001 C CNN
+F 3 "~" H 1675 8725 50  0001 C CNN
+	1    1675 8725
+	-1   0    0    -1
+$EndComp
+Text GLabel 1850 8125 0    55   Input ~ 0
+12V
+Wire Wire Line
+	1750 8525 1675 8525
+Wire Wire Line
+	1675 8525 1675 8575
+Wire Wire Line
+	1675 8525 1225 8525
+Connection ~ 1675 8525
+Connection ~ 1225 8525
+Wire Wire Line
+	1675 8875 1675 8925
+Connection ~ 1675 8925
+Wire Wire Line
+	1950 8725 1950 8925
+Wire Wire Line
+	1675 8925 1950 8925
+Connection ~ 1950 8925
+Wire Wire Line
+	1950 8925 1950 8975
+Wire Wire Line
+	2000 8125 1850 8125
+Wire Wire Line
+	1950 8225 1950 8325
 Wire Notes Line
-	2475 8850 875  8850
+	2475 7750 2475 9150
 Wire Notes Line
-	875  8850 875  7750
+	875  7750 875  9150
 $EndSCHEMATC
