File: pcb/main/3.kicad_sch (KiCad schematic)
At the start: 12 parts, among them U3 ACT4088

Commit message: Add fields to PCBA
Parts:
- C12: value 22nF -> 22n
- C13: value 10µF -> 10u; MFN (none) -> Samsung Electro-Mechanics; MFP (none) -> CL21A106KOQNNNG; S1PL (none) -> https://www.mouser.com/ProductDetail/Samsung-Electro-Mechan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; S1PN (none) -> 187-CL21A106KOQNNNG
- C14: value 22µF -> 22u
- L1: value 4.7µH -> 4.7u
Changed lines of the file:
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@@
     (in_bom yes) (on_board yes)
     (property "Reference" "L1" (id 0) (at 130.175 98.425 90))
-    (property "Value" "4.7µH" (id 1) (at 130.175 101.6 90))
+    (property "Value" "4.7u" (id 1) (at 130.175 101.6 90))
     (property "Footprint" "Inductor_SMD:L_0805_2012Metric_Pad1.15x1.40mm_HandSolder" (id 2) (at 130.175 100.33 0)
       (effects (font (size 1.27 1.27)) hide)
@@
     )
   )
-  (symbol (lib_id "Device:R") (at 211.455 92.075 270)
+  (symbol (lib_id "Device:R") (at 211.455 92.075 270) (unit 1)
     (in_bom yes) (on_board yes)
     (property "Reference" "R22" (id 0) (at 211.455 90.17 90))
@@
     )
   )
-  (symbol (lib_id "Device:R") (at 211.455 107.315 270)
+  (symbol (lib_id "Device:R") (at 211.455 107.315 270) (unit 1)
     (in_bom yes) (on_board yes)
     (property "Reference" "R23" (id 0) (at 211.455 105.41 90))
@@
       (effects (font (size 1.27 1.27)) (justify left))
     )
-    (property "Value" "10µF" (id 1) (at 98.806 100.203 0)
+    (property "Value" "10u" (id 1) (at 98.806 100.203 0)
       (effects (font (size 1.27 1.27)) (justify left))
     )
@@
       (effects (font (size 1.27 1.27)) hide)
     )
-    (property "Datasheet" "~" (id 3) (at 95.885 99.06 0)
+    (property "Datasheet" "https://www.mouser.com/datasheet/2/585/MLCC-1837944.pdf" (id 3) (at 95.885 99.06 0)
+      (effects (font (size 1.27 1.27)) hide)
+    )
+    (property "MFN" "Samsung Electro-Mechanics " (id 4) (at 95.885 99.06 0)
+      (effects (font (size 1.27 1.27)) hide)
+    )
+    (property "MFP" "CL21A106KOQNNNG " (id 5) (at 95.885 99.06 0)
+      (effects (font (size 1.27 1.27)) hide)
+    )
+    (property "S1PL" "https://www.mouser.com/ProductDetail/Samsung-Electro-Mechanics/CL21A106KOQNNNG?qs=hqM3L16%252BxlcMWI7QbqH0LA%3D%3D" (id 6) (at 95.885 99.06 0)
+      (effects (font (size 1.27 1.27)) hide)
+    )
+    (property "S1PN" " 187-CL21A106KOQNNNG " (id 7) (at 95.885 99.06 0)
+      (effects (font (size 1.27 1.27)) hide)
+    )
+    (property "Description" "Multilayer Ceramic Capacitors MLCC - SMD/SMT 16V 10uF XX5R 0805 10%" (id 4) (at 95.885 99.06 0)
       (effects (font (size 1.27 1.27)) hide)
     )
@@
       (effects (font (size 1.27 1.27)) (justify left))
     )
-    (property "Value" "22nF" (id 1) (at 124.206 96.393 0)
+    (property "Value" "22n" (id 1) (at 124.206 96.393 0)
       (effects (font (size 1.27 1.27)) (justify left))
     )
@@
       (effects (font (size 1.27 1.27)) (justify left))
     )
-    (property "Value" "22µF" (id 1) (at 144.526 106.553 0)
+    (property "Value" "22u" (id 1) (at 144.526 106.553 0)
       (effects (font (size 1.27 1.27)) (justify left))
     )

Commit message: Update 2: Fields for BOM with PCBA manufacturer
Parts:
- C12: MFN (none) -> Wurth Elektronik; MFP (none) -> 885012207094; S1PL (none) -> https://www.mouser.com/ProductDetail/Wurth-Elektronik/88501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; S1PN (none) -> 710-885012207094
- C14: MFN (none) -> Samsung Electro-Mechanics; MFP (none) -> CL21A226KQCLRNC; S1PL (none) -> https://www.mouser.com/ProductDetail/Samsung-Electro-Mechan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; S1PN (none) -> 187-CL21A226KQCLRNC
- D11, D13: MFN (none) -> Wurth Elektronik; MFP (none) -> 150080GS75000; S1PL (none) -> https://www.mouser.com/ProductDetail/Wurth-Elektronik/15008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; S1PN (none) -> 710-150080GS75000
- D12: footprint Diode_SMD:D_SOD-123 -> Diode_SMD:D_SMA; MFN (none) -> Vishay Semiconductors; MFP (none) -> B240A-E3/61T; S1PL (none) -> https://www.mouser.com/ProductDetail/Vishay-Semiconductors/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; S1PN (none) -> 625-B240A-E3/61T
- L1: MFN (none) -> Taiyo Yuden; MFP (none) -> CKP2012N4R7M-T; S1PL (none) -> https://www.mouser.com/ProductDetail/Taiyo-Yuden/CKP2012N4R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; S1PN (none) -> 963-CKP2012N4R7M-T
Other:
- note added: "The inductor's DC resistance should be less than 250 mΩ. The input capacitor, electrolytic, or ceramics with low ESR should be used."
Changed lines of the file:
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@@
     (stroke (width 0) (type solid) (color 0 0 0 0))
+  )
+  (text "The inductor's DC resistance should be less than 250 mΩ.\n\nThe  input  capacitor,  electrolytic,  or  ceramics  with  low  ESR\nshould  be  used."
+    (at 86.4616 137.9474 0)
+    (effects (font (size 1.27 1.27)) (justify left bottom))
   )
   (text "3.3v: 16.23k\n5v: 9.64k" (at 125.095 124.46 0)
@@
       (effects (font (size 1.27 1.27)) hide)
     )
-    (property "Datasheet" "~" (id 3) (at 130.175 100.33 0)
+    (property "Datasheet" "https://www.mouser.com/datasheet/2/396/mlci03_e-1523425.pdf" (id 3) (at 130.175 100.33 0)
+      (effects (font (size 1.27 1.27)) hide)
+    )
+    (property "Description" "Fixed Inductors 0805 4.7uH 280mOhms +/-20% 700mA HiCur" (id 4) (at 130.175 100.33 0)
+      (effects (font (size 1.27 1.27)) hide)
+    )
+    (property "MFN" "Taiyo Yuden " (id 5) (at 130.175 100.33 0)
+      (effects (font (size 1.27 1.27)) hide)
+    )
+    (property "MFP" "CKP2012N4R7M-T" (id 6) (at 130.175 100.33 0)
+      (effects (font (size 1.27 1.27)) hide)
+    )
+    (property "S1PL" "https://www.mouser.com/ProductDetail/Taiyo-Yuden/CKP2012N4R7M-T?qs=I6KAKw0tg2yv0trrzbAvhA%3D%3D" (id 7) (at 130.175 100.33 0)
+      (effects (font (size 1.27 1.27)) hide)
+    )
+    (property "S1PN" " 963-CKP2012N4R7M-T " (id 8) (at 130.175 100.33 0)
       (effects (font (size 1.27 1.27)) hide)
     )
@@
       (effects (font (size 1.27 1.27)) (justify left))
     )
-    (property "Footprint" "Diode_SMD:D_SOD-123" (id 2) (at 121.285 104.14 0)
+    (property "Footprint" "Diode_SMD:D_SMA" (id 2) (at 121.285 104.14 0)
       (effects (font (size 1.27 1.27)) hide)
     )
     (property "Datasheet" "~" (id 3) (at 121.285 104.14 0)
+      (effects (font (size 1.27 1.27)) hide)
+    )
+    (property "Description" "Schottky Diodes & Rectifiers 2.0 Amp 40 Volt " (id 4) (at 121.285 104.14 0)
+      (effects (font (size 1.27 1.27)) hide)
+    )
+    (property "MFN" "Vishay Semiconductors " (id 5) (at 121.285 104.14 0)
+      (effects (font (size 1.27 1.27)) hide)
+    )
+    (property "MFP" "B240A-E3/61T" (id 6) (at 121.285 104.14 0)
+      (effects (font (size 1.27 1.27)) hide)
+    )
+    (property "S1PL" "https://www.mouser.com/ProductDetail/Vishay-Semiconductors/B240A-E3-61T?qs=tdXsjSi%2FIMZoZjTYxlkTBQ%3D%3D" (id 7) (at 121.285 104.14 0)
+      (effects (font (size 1.27 1.27)) hide)
+    )
+    (property "S1PN" " 625-B240A-E3/61T " (id 8) (at 121.285 104.14 0)
       (effects (font (size 1.27 1.27)) hide)
     )
@@
       (effects (font (size 1.27 1.27)) hide)
     )
+    (property "Description" "Standard LEDs - SMD WL-SMCW SMDMono TpVw Waterclr 0805 Green " (id 4) (at 188.595 92.075 0)
+      (effects (font (size 1.27 1.27)) hide)
+    )
+    (property "MFN" "Wurth Elektronik " (id 5) (at 188.595 92.075 0)
+      (effects (font (size 1.27 1.27)) hide)
+    )
+    (property "MFP" "150080GS75000 " (id 6) (at 188.595 92.075 0)
+      (effects (font (size 1.27 1.27)) hide)
+    )
+    (property "S1PL" "https://www.mouser.com/ProductDetail/Wurth-Elektronik/150080GS75000?qs=2kOmHSv6VfQRoTEZVk1mGA%3D%3D" (id 7) (at 188.595 92.075 0)
+      (effects (font (size 1.27 1.27)) hide)
+    )
+    (property "S1PN" " 710-150080GS75000 " (id 8) (at 188.595 92.075 0)
+      (effects (font (size 1.27 1.27)) hide)
+    )
   )
   (symbol (lib_id "Device:LED") (at 188.595 107.315 0) (mirror x) (unit 1)
@@
       (effects (font (size 1.27 1.27)) hide)
     )
+    (property "Description" "Standard LEDs - SMD WL-SMCW SMDMono TpVw Waterclr 0805 Green " (id 4) (at 188.595 107.315 0)
+      (effects (font (size 1.27 1.27)) hide)
+    )
+    (property "MFN" "Wurth Elektronik " (id 5) (at 188.595 107.315 0)
+      (effects (font (size 1.27 1.27)) hide)
+    )
+    (property "MFP" "150080GS75000 " (id 6) (at 188.595 107.315 0)
+      (effects (font (size 1.27 1.27)) hide)
+    )
+    (property "S1PL" "https://www.mouser.com/ProductDetail/Wurth-Elektronik/150080GS75000?qs=2kOmHSv6VfQRoTEZVk1mGA%3D%3D" (id 7) (at 188.595 107.315 0)
+      (effects (font (size 1.27 1.27)) hide)
+    )
+    (property "S1PN" " 710-150080GS75000 " (id 8) (at 188.595 107.315 0)
+      (effects (font (size 1.27 1.27)) hide)
+    )
   )
   (symbol (lib_id "Device:C") (at 95.885 99.06 0) (unit 1)
@@
       (effects (font (size 1.27 1.27)) hide)
     )
-    (property "Description" "Multilayer Ceramic Capacitors MLCC - SMD/SMT 16V 10uF XX5R 0805 10%" (id 4) (at 95.885 99.06 0)
+    (property "Description" "Multilayer Ceramic Capacitors MLCC - SMD/SMT 16V 10uF X5R 0805 10%" (id 4) (at 95.885 99.06 0)
       (effects (font (size 1.27 1.27)) hide)
     )
@@
       (effects (font (size 1.27 1.27)) hide)
     )
+    (property "Description" "Multilayer Ceramic Capacitors MLCC - SMD/SMT 50V WCAP-CSGP 0.022uF 0805 10% MLCC " (id 4) (at 121.285 95.25 0)
+      (effects (font (size 1.27 1.27)) hide)
+    )
+    (property "MFN" "Wurth Elektronik " (id 5) (at 121.285 95.25 0)
+      (effects (font (size 1.27 1.27)) hide)
+    )
+    (property "MFP" "885012207094 " (id 6) (at 121.285 95.25 0)
+      (effects (font (size 1.27 1.27)) hide)
+    )
+    (property "S1PL" "https://www.mouser.com/ProductDetail/Wurth-Elektronik/885012207094?qs=0KOYDY2FL2868KFEJBLp3w%3D%3D" (id 7) (at 121.285 95.25 0)
+      (effects (font (size 1.27 1.27)) hide)
+    )
+    (property "S1PN" " 710-885012207094 " (id 8) (at 121.285 95.25 0)
+      (effects (font (size 1.27 1.27)) hide)
+    )
   )
   (symbol (lib_id "Device:C") (at 141.605 105.41 0) (unit 1)
@@
       (effects (font (size 1.27 1.27)) hide)
     )
+    (property "Description" "Multilayer Ceramic Capacitors MLCC - SMD/SMT 6.3V 22uF X5R 10% 0805" (id 4) (at 141.605 105.41 0)
+      (effects (font (size 1.27 1.27)) hide)
+    )
+    (property "MFN" "Samsung Electro-Mechanics " (id 5) (at 141.605 105.41 0)
+      (effects (font (size 1.27 1.27)) hide)
+    )
+    (property "MFP" "CL21A226KQCLRNC" (id 6) (at 141.605 105.41 0)
+      (effects (font (size 1.27 1.27)) hide)
+    )
+    (property "S1PL" "https://www.mouser.com/ProductDetail/Samsung-Electro-Mechanics/CL21A226KQCLRNC?qs=xZ%2FP%252Ba9zWqYG0ePGTF%2FymQ%3D%3D" (id 7) (at 141.605 105.41 0)
+      (effects (font (size 1.27 1.27)) hide)
+    )
+    (property "S1PN" " 187-CL21A226KQCLRNC " (id 8) (at 141.605 105.41 0)
+      (effects (font (size 1.27 1.27)) hide)
+    )

Commit message: Update 3 - BOM for PCBA
Parts:
- R22: MFN (none) -> KOA Speer; MFP (none) -> RK73H2ATTD1002F; S1PL (none) -> https://www.mouser.com/ProductDetail/KOA-Speer/RK73H2ATTD10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; S1PN (none) -> 660-RK73H2ATTD1002F
- R23: MFN (none) -> Vishay / Dale; MFP (none) -> CRCW08051K00JNEAC; S1PL (none) -> https://www.mouser.com/ProductDetail/Vishay-Dale/CRCW08051K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; S1PN (none) -> 71-CRCW08051K00JNEAC
- R24: MFN (none) -> KOA Speer; MFP (none) -> RK73H2ATTD4992F; S1PL (none) -> https://www.mouser.com/ProductDetail/KOA-Speer/RK73H2ATTD49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; S1PN (none) -> 660-RK73H2ATTD4992F
- R25: MFN (none) -> Panasonic; MFP (none) -> ERJ-6ENF1622V; S1PL (none) -> https://www.mouser.com/ProductDetail/Panasonic/ERJ-6ENF1622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; S1PN (none) -> 667-ERJ-6ENF1622V
- U3: MFN (none) -> Qorvo; MFP (none) -> ACT4088US-T; S1PL (none) -> https://www.mouser.com/ProductDetail/Qorvo/ACT4088US-T?qs=%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; S1PN (none) -> 107-ACT4088US-T
Changed lines of the file:
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@@
   (junction (at 141.605 100.33) (diameter 1.016) (color 0 0 0 0))
   (junction (at 176.53 99.06) (diameter 1.016) (color 0 0 0 0))
+  (no_connect (at 64.135 54.61))
   (no_connect (at 102.235 105.41))
-  (no_connect (at 64.135 54.61))
   (wire (pts (xy 94.615 93.98) (xy 95.885 93.98))
     (stroke (width 0) (type solid) (color 0 0 0 0))
@@
       (effects (font (size 1.27 1.27)) hide)
     )
-    (property "Datasheet" "~" (id 3) (at 121.285 116.84 0)
+    (property "Datasheet" "https://www.mouser.com/datasheet/2/315/AOA0000C304-1149620.pdf" (id 3) (at 121.285 116.84 0)
+      (effects (font (size 1.27 1.27)) hide)
+    )
+    (property "Description" "Thick Film Resistors - SMD 0805 16.2Kohms 1% AEC-Q200" (id 4) (at 121.285 116.84 0)
+      (effects (font (size 1.27 1.27)) hide)
+    )
+    (property "MFN" "Panasonic " (id 5) (at 121.285 116.84 0)
+      (effects (font (size 1.27 1.27)) hide)
+    )
+    (property "MFP" "ERJ-6ENF1622V" (id 6) (at 121.285 116.84 0)
+      (effects (font (size 1.27 1.27)) hide)
+    )
+    (property "S1PL" "https://www.mouser.com/ProductDetail/Panasonic/ERJ-6ENF1622V?qs=sGAEpiMZZMtlubZbdhIBINbsJb0hdM3zKmmABjaHwtM%3D" (id 7) (at 121.285 116.84 0)
+      (effects (font (size 1.27 1.27)) hide)
+    )
+    (property "S1PN" " 667-ERJ-6ENF1622V " (id 8) (at 121.285 116.84 0)
       (effects (font (size 1.27 1.27)) hide)
     )
@@
       (effects (font (size 1.27 1.27)) hide)
     )
-    (property "Datasheet" "~" (id 3) (at 130.175 110.49 0)
+    (property "Datasheet" "https://www.mouser.com/datasheet/2/219/RK73H-1825326.pdf" (id 3) (at 130.175 110.49 0)
+      (effects (font (size 1.27 1.27)) hide)
+    )
+    (property "Description" "Thick Film Resistors - SMD .125watt 49.9kohms 1% 0805 100ppm" (id 4) (at 130.175 110.49 0)
+      (effects (font (size 1.27 1.27)) hide)
+    )
+    (property "MFN" "KOA Speer " (id 5) (at 130.175 110.49 0)
+      (effects (font (size 1.27 1.27)) hide)
+    )
+    (property "MFP" "RK73H2ATTD4992F " (id 6) (at 130.175 110.49 0)
+      (effects (font (size 1.27 1.27)) hide)
+    )
+    (property "S1PL" "https://www.mouser.com/ProductDetail/KOA-Speer/RK73H2ATTD4992F?qs=sGAEpiMZZMtlubZbdhIBIPHHA4tSuOuyusuxPBWaS8c%3D" (id 7) (at 130.175 110.49 0)
+      (effects (font (size 1.27 1.27)) hide)
+    )
+    (property "S1PN" " 660-RK73H2ATTD4992F " (id 8) (at 130.175 110.49 0)
       (effects (font (size 1.27 1.27)) hide)
     )
@@
       (effects (font (size 1.27 1.27)) hide)
     )
-    (property "Datasheet" "~" (id 3) (at 211.455 92.075 0)
+    (property "Datasheet" "https://www.mouser.com/datasheet/2/219/RK73H-1825326.pdf" (id 3) (at 211.455 92.075 0)
+      (effects (font (size 1.27 1.27)) hide)
+    )
+    (property "Description" "Thick Film Resistors - SMD 1/4W 10K OHM 1%" (id 4) (at 211.455 92.075 0)
+      (effects (font (size 1.27 1.27)) hide)
+    )
+    (property "MFN" "KOA Speer " (id 5) (at 211.455 92.075 0)
+      (effects (font (size 1.27 1.27)) hide)
+    )
+    (property "MFP" "RK73H2ATTD1002F" (id 6) (at 211.455 92.075 0)
+      (effects (font (size 1.27 1.27)) hide)
+    )
+    (property "S1PL" "https://www.mouser.com/ProductDetail/KOA-Speer/RK73H2ATTD1002F?qs=sGAEpiMZZMtlubZbdhIBIADEshVnklemK%252BhrLNEuMe8%3D" (id 7) (at 211.455 92.075 0)
+      (effects (font (size 1.27 1.27)) hide)
+    )
+    (property "S1PN" " 660-RK73H2ATTD1002F " (id 8) (at 211.455 92.075 0)
       (effects (font (size 1.27 1.27)) hide)
     )
@@
       (effects (font (size 1.27 1.27)) hide)
     )
-    (property "Datasheet" "~" (id 3) (at 211.455 107.315 0)
+    (property "Datasheet" "https://www.mouser.com/datasheet/2/427/crcwce3-1762584.pdf" (id 3) (at 211.455 107.315 0)
+      (effects (font (size 1.27 1.27)) hide)
+    )
+    (property "Description" "Thick Film Resistors - SMD 1/8Watt 1Kohms 5% Commercial Use" (id 4) (at 211.455 107.315 0)
+      (effects (font (size 1.27 1.27)) hide)
+    )
+    (property "MFN" "Vishay / Dale " (id 5) (at 211.455 107.315 0)
+      (effects (font (size 1.27 1.27)) hide)
+    )
+    (property "MFP" "CRCW08051K00JNEAC " (id 6) (at 211.455 107.315 0)
+      (effects (font (size 1.27 1.27)) hide)
+    )
+    (property "S1PL" "https://www.mouser.com/ProductDetail/Vishay-Dale/CRCW08051K00JNEAC?qs=sGAEpiMZZMtlubZbdhIBIIZe04wfiaJWy7nwcSDiXks%3D" (id 7) (at 211.455 107.315 0)
+      (effects (font (size 1.27 1.27)) hide)
+    )
+    (property "S1PN" " 71-CRCW08051K00JNEAC " (id 8) (at 211.455 107.315 0)
       (effects (font (size 1.27 1.27)) hide)
     )
@@
       (effects (font (size 1.27 1.27)) hide)
     )
-    (property "Datasheet" "" (id 3) (at 111.125 101.6 0)
-      (effects (font (size 1.27 1.27)) hide)
-    )
+    (property "Datasheet" "https://www.mouser.com/datasheet/2/412/ACT4088_Data_Sheet-1714846.pdf" (id 3) (at 111.125 101.6 0)
+      (effects (font (size 1.27 1.27)) hide)
+    )
+    (property "Description" "Switching Voltage Regulators DC70DZUST, 12Vin Buck Converter " (id 4) (at 109.855 101.6 0)
+      (effects (font (size 1.27 1.27)) hide)
+    )
+    (property "MFN" "Qorvo " (id 5) (at 109.855 101.6 0)
+      (effects (font (size 1.27 1.27)) hide)
+    )
+    (property "MFP" "ACT4088US-T" (id 6) (at 109.855 101.6 0)
+      (effects (font (size 1.27 1.27)) hide)
+    )
+    (property "S1PL" "https://www.mouser.com/ProductDetail/Qorvo/ACT4088US-T?qs=%2Fha2pyFaduj3zC6esU%2F8%252BfzWZ4716qD%252Byca2A%252BeLaTI%3D" (id 7) (at 109.855 101.6 0)
+      (effects (font (size 1.27 1.27)) hide)
+    )
+    (property "S1PN" " 107-ACT4088US-T " (id 8) (at 109.855 101.6 0)
+      (effects (font (size 1.27 1.27)) hide)
+    )

Commit message: Update 5 - BOM for PCBA. Check 1 issue #46
Parts:
- removed D12: B240A, Diode_SMD:D_SMA, symbol Device:D
- added D12: MBR0520LT1G, Diode_SMD:D_SOD-123, symbol Device:D_Schottky
Connections:
- net GND: now also D12.2 (A)
- net at C12.2, L1.1, U3.1 (SW): now also D12.1 (K)
Changed lines of the file:
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@@
     )
   )
-  (symbol (lib_id "Device:D") (at 121.285 104.14 270) (unit 1)
+  (symbol (lib_id "Device:D_Schottky") (at 121.285 104.14 270) (unit 1)
     (in_bom yes) (on_board yes)
-    (property "Reference" "D12" (id 0) (at 123.2916 102.9716 90)
-      (effects (font (size 1.27 1.27)) (justify left))
-    )
-    (property "Value" "B240A" (id 1) (at 123.2916 105.283 90)
-      (effects (font (size 1.27 1.27)) (justify left))
-    )
-    (property "Footprint" "Diode_SMD:D_SMA" (id 2) (at 121.285 104.14 0)
+    (property "Reference" "D12" (id 0) (at 123.825 104.14 0))
+    (property "Value" "MBR0520LT1G " (id 1) (at 119.38 103.505 0))
+    (property "Footprint" "Diode_SMD:D_SOD-123" (id 2) (at 121.285 104.14 0)
       (effects (font (size 1.27 1.27)) hide)
     )
-    (property "Datasheet" "~" (id 3) (at 121.285 104.14 0)
+    (property "Datasheet" "https://www.mouser.com/datasheet/2/308/MBR0520LT1_D-1810808.pdf" (id 3) (at 121.285 104.14 0)
       (effects (font (size 1.27 1.27)) hide)
     )
-    (property "Description" "Schottky Diodes & Rectifiers 2.0 Amp 40 Volt " (id 4) (at 121.285 104.14 0)
+    (property "Description" "Schottky Diodes & Rectifiers 0.5A 20V " (id 4) (at 121.285 104.14 0)
       (effects (font (size 1.27 1.27)) hide)
     )
-    (property "MFN" "Vishay Semiconductors " (id 5) (at 121.285 104.14 0)
+    (property "MFN" "ON Semiconductor " (id 5) (at 121.285 104.14 0)
       (effects (font (size 1.27 1.27)) hide)
     )
-    (property "MFP" "B240A-E3/61T" (id 6) (at 121.285 104.14 0)
+    (property "MFP" "MBR0520LT1G " (id 6) (at 121.285 104.14 0)
       (effects (font (size 1.27 1.27)) hide)
     )
-    (property "S1PL" "https://www.mouser.com/ProductDetail/Vishay-Semiconductors/B240A-E3-61T?qs=tdXsjSi%2FIMZoZjTYxlkTBQ%3D%3D" (id 7) (at 121.285 104.14 0)
+    (property "S1PL" "https://www.mouser.com/ProductDetail/ON-Semiconductor/MBR0520LT1G?qs=3JMERSakebqBWTiPUQp0nw%3D%3D" (id 7) (at 121.285 104.14 0)
       (effects (font (size 1.27 1.27)) hide)
     )
-    (property "S1PN" " 625-B240A-E3/61T " (id 8) (at 121.285 104.14 0)
+    (property "S1PN" " 863-MBR0520LT1G " (id 8) (at 121.285 104.14 0)
       (effects (font (size 1.27 1.27)) hide)
     )
@@
       (effects (font (size 1.27 1.27)) hide)
     )
-    (property "Datasheet" "~" (id 3) (at 188.595 92.075 0)
+    (property "Datasheet" "https://www.mouser.com/datasheet/2/445/150080GS75000-1715657.pdf" (id 3) (at 188.595 92.075 0)
       (effects (font (size 1.27 1.27)) hide)
     )
@@
       (effects (font (size 1.27 1.27)) hide)
     )
-    (property "Datasheet" "~" (id 3) (at 188.595 107.315 0)
+    (property "Datasheet" "https://www.mouser.com/datasheet/2/445/150080GS75000-1715657.pdf" (id 3) (at 188.595 107.315 0)
       (effects (font (size 1.27 1.27)) hide)
     )
@@
       (effects (font (size 1.27 1.27)) hide)
     )
-    (property "Datasheet" "~" (id 3) (at 121.285 95.25 0)
+    (property "Datasheet" "https://www.mouser.com/datasheet/2/445/885012207094-1727634.pdf" (id 3) (at 121.285 95.25 0)
       (effects (font (size 1.27 1.27)) hide)
     )
@@
       (effects (font (size 1.27 1.27)) hide)
     )
-    (property "Datasheet" "~" (id 3) (at 141.605 105.41 0)
+    (property "Datasheet" "https://www.mouser.com/datasheet/2/585/MLCC-1837944.pdf" (id 3) (at 141.605 105.41 0)
       (effects (font (size 1.27 1.27)) hide)
     )
