File: pcb/main/Bertha_main.kicad_sch (KiCad schematic)
At the start: 87 parts, among them J1 RJ12, J12 AudioJack3_SwitchTR, J2 Conn_Coaxial_Power, J3 Conn_02x03_Odd_Even, J4 RJ12, J5 AudioJack3_SwitchTR, J6 SJ, J7 Conn_01x01, J8 Conn_01x01, Q1 ZXMS6004, Q2 ZXMS6004, Q3 IPB80N03S4L-03, Q5 ZXMS6004, Q6 ZXMS6004, Q7 ZXMS6004, Q8 ZXMS6004, U1 DS18B20, U2 ATMEGA32U4-AU, X1 MINI-USB-SCHIELD-32005-201, Y1 Crystal

Commit message: Add fields to PCBA
Parts:
- C1, C3, C4: value 10uF -> 10u; MFN (none) -> Samsung Electro-Mechanics; MFP (none) -> CL21A106KOQNNNG; S1PL (none) -> https://www.mouser.com/ProductDetail/Samsung-Electro-Mechan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; S1PN (none) -> 187-CL21A106KOQNNNG
- C10, C9: value 22pF -> 22p; MFN (none) -> AVX; MFP (none) -> 08055A220JAT2A; S1PL (none) -> https://www.mouser.com/ProductDetail/AVX/08055A220JAT2A?qs=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; S1PN (none) -> 581-08055A220J
- C11, C2, C34, C35, C38, C5, C6, C7, C8: value 100nF -> 100n; MFN (none) -> Samsung Electro-Mechanics; MFP (none) -> CL21A106KOQNNNG; S1PL (none) -> https://www.mouser.com/ProductDetail/Samsung-Electro-Mechan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; S1PN (none) -> 187-CL21A106KOQNNNG
- J2: MFN (none) -> SparkFun; MFP (none) -> PRT-00119; S1PL (none) -> https://www.mouser.com/ProductDetail/SparkFun/PRT-00119?qs=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; S1PN (none) -> 474-PRT-00119
- Q1: MFP (none) -> ZXMS6004FFTA; MFR ZXMS6004FFTA -> (none); Mouser 522-ZXMS6004FFTA -> (none); S1PN (none) -> 522-ZXMS6004FFTA

Commit message: Update 2: Fields for BOM with PCBA manufacturer
Parts:
- C10, C9: footprint Capacitor_SMD:C_1206_3216Metric_Pad1.42x1.75mm_HandSolder -> Capacitor_SMD:C_0805_2012Metric_Pad1.18x1.45mm_HandSolder
- D1, D2, D3: value D_Schottky -> MBR0520LT1G; MFN (none) -> ON Semiconductor; MFP (none) -> MBR0520LT1G; S1PL (none) -> https://www.mouser.com/ProductDetail/ON-Semiconductor/MBR05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; S1PN (none) -> 863-MBR0520LT1G
- D10, D20, D21: MFN (none) -> Wurth Elektronik; MFP (none) -> 150080SS75000; S1PL (none) -> https://www.mouser.com/ProductDetail/Wurth-Elektronik/15008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; S1PN (none) -> 710-150080SS75000
- D18, D19, D8, D9: MFN (none) -> Wurth Elektronik; MFP (none) -> 150080BS75000; S1PL (none) -> https://www.mouser.com/ProductDetail/Wurth-Elektronik/15008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; S1PN (none) -> 710-150080BS75000
- D4, D5, D7: MFN (none) -> Wurth Elektronik; MFP (none) -> 150080YS75000; S1PL (none) -> https://www.mouser.com/ProductDetail/Wurth-Elektronik/15008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; S1PN (none) -> 710-150080YS75000
- D6: value WHITE -> GREEN; MFN (none) -> Wurth Elektronik; MFP (none) -> 150080GS75000; S1PL (none) -> https://www.mouser.com/ProductDetail/Wurth-Elektronik/15008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; S1PN (none) -> 710-150080GS75000
- J1, J4: MFN (none) -> Pulse Electronics; MFP (none) -> E5566-Q0LK22-L; S1PL (none) -> https://www.mouser.com/ProductDetail/Pulse-Electronics/E556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; S1PN (none) -> 673-E5566-Q0LK22-L
- JP1, JP2: MFN (none) -> Molex; MFP (none) -> 22-28-4020; S1PL (none) -> https://www.mouser.com/ProductDetail/Molex/22-28-4020?qs=d9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; S1PN (none) -> 538-22-28-4020
- JP13, JP14, JP3, JP4, JP8, JP9: MFN (none) -> Molex; MFP (none) -> 22-23-2023; S1PL (none) -> https://www.mouser.com/ProductDetail/Molex/22-23-2023?qs=52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; S1PN (none) -> 538-22-23-2023
- Q1: MFN (none) -> Diodes Incorporated; MFP ZXMS6004FFTA -> ZXMS6004FFQTA; S1PL (none) -> https://www.mouser.com/ProductDetail/Diodes-Incorporated/ZX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; S1PN 522-ZXMS6004FFTA -> 621-ZXMS6004FFQTA
- Q2, Q5, Q6, Q7: MFN (none) -> Diodes Incorporated; MFP (none) -> ZXMS6004FFQTA; S1PL (none) -> https://www.mouser.com/ProductDetail/Diodes-Incorporated/ZX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; S1PN (none) -> 621-ZXMS6004FFQTA
- Q3: MFN (none) -> Infineon Technologies; MFP (none) -> IPB80N03S4L-03; S1PL (none) -> https://www.mouser.com/ProductDetail/Infineon-Technologies/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; S1PN (none) -> 726-IPB80N03S4L-03
- Q8: MFN (none) -> Diodes Incorporated; MFP ZXMS6004FFTA -> ZXMS6004FFQTA; S1PL (none) -> https://www.mouser.com/ProductDetail/Diodes-Incorporated/ZX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; S1PN (none) -> 621-ZXMS6004FFQTA

Commit message: Update 3 - BOM for PCBA
Parts:
- R1, R10, R15, R17, R2, R20, R21, R52, R53, R54, R55: MFN (none) -> KOA Speer; MFP (none) -> RK73H2ATTD1002F; S1PL (none) -> https://www.mouser.com/ProductDetail/KOA-Speer/RK73H2ATTD10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; S1PN (none) -> 660-RK73H2ATTD1002F
- R11, R13, R14, R16, R51, R7, R9: MFN (none) -> Vishay / Dale; MFP (none) -> CRCW08051K00JNEAC; S1PL (none) -> https://www.mouser.com/ProductDetail/Vishay-Dale/CRCW08051K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; S1PN (none) -> 71-CRCW08051K00JNEAC
- R12, R50, R6: MFN (none) -> KOA Speer; MFP (none) -> RK73H2ATTD4701F; S1PL (none) -> https://www.mouser.com/ProductDetail/KOA-Speer/RK73H2ATTD47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; S1PN (none) -> 660-RK73H2ATTD4701F
- R18: MFN (none) -> Vishay / Dale; MFP (none) -> CRCW08051M00FKEAC; S1PL (none) -> https://www.mouser.com/ProductDetail/Vishay-Dale/CRCW08051M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; S1PN (none) -> 71-CRCW08051M00FKEAC
- R19, R5, R8: MFN (none) -> Bourns; MFP (none) -> CMP0805-FX-1000ELF; S1PL (none) -> https://www.mouser.com/ProductDetail/Bourns/CMP0805-FX-1000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; S1PN (none) -> 652-CMP0805-FX-1000L
- R3, R4: MFN (none) -> Vishay / Dale; MFP (none) -> CRCW080522R0FKEAC; S1PL (none) -> https://www.mouser.com/ProductDetail/Vishay-Dale/CRCW080522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; S1PN (none) -> 71-CRCW080522R0FKEAC
- U1: MFN (none) -> Maxim Integrated; MFP (none) -> DS18B20U+T&R; S1PL (none) -> https://www.mouser.com/ProductDetail/Maxim-Integrated/DS18B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; S1PN (none) -> 700-DS18B20UT&R
- U2: MFN (none) -> Microchip Technology / Atmel; MFP (none) -> ATMEGA32U4RC-AU; S1PL (none) -> https://www.mouser.com/ProductDetail/Microchip-Technology-A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; S1PN (none) -> 556-ATMEGA32U4RC-AU
- X1: MFN (none) -> Molex; MFP (none) -> 67503-1020; S1PL (none) -> https://www.mouser.com/ProductDetail/Molex/67503-1020?qs=7z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; S1PN (none) -> 538-67503-1020
- Y1: MFN (none) -> ECS; MFP (none) -> ECS-80-18-23B-JTM-TR; S1PL (none) -> https://www.mouser.com/ProductDetail/ECS/ECS-80-18-23B-JTM-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; S1PN (none) -> 520-80-18-23B-JTMT

Commit message: Update 4 - BOM for PCBA. Ready  to check issue #46
Parts:
- C11, C2, C34, C35, C38, C5, C6, C7, C8: MFN Samsung Electro-Mechanics -> AVX; MFP CL21A106KOQNNNG -> 08055C104KAT2A; S1PL https://www.mouser.com/ProductDetail/Samsung-Electro-Mechan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 -> https://www.mouser.com/ProductDetail/AVX/08055C104KAT2A?qs=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; S1PN 187-CL21A106KOQNNNG -> 581-08055C104K
- J12, J5: S1PL (none) -> https://www.aliexpress.com/item/33004214640.html?spm=a2g0s.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

Commit message: Update 5 - BOM for PCBA. Check 1 issue #46
Parts:
- Y1: MFP ECS-80-18-23B-JTM-TR -> ECS-080-18-23G-JGN-TR; S1PL https://www.mouser.com/ProductDetail/ECS/ECS-80-18-23B-JTM-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 -> https://www.mouser.com/ProductDetail/ECS/ECS-080-18-23G-JGN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; S1PN 520-80-18-23B-JTMT -> 520-8.0-18-23G-JGNT

Commit message: Update UCAP for uC 100n -> 1u
Parts:
- C8: value 100n -> 1u

Commit message: Fix: capacitors value for crystal (22p to 18 p)
Parts:
- C10, C9: value 22p -> 18p; MFN AVX -> KEMET; MFP 08055A220JAT2A -> C0805C180K5HACTU; S1PL https://www.mouser.com/ProductDetail/AVX/08055A220JAT2A?qs=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 -> https://www.mouser.com/ProductDetail/KEMET/C0805C180K5HACTU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; S1PN 581-08055A220J -> 80-C0805C180K5HACTU
Changed lines of the file:
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@@
-(kicad_sch (version 20200828) (generator eeschema)
+(kicad_sch (version 20201015) (generator eeschema)
   (page 1 5)
   (paper "A3")
