File: pcb/main/Flash Memory.kicad_sch (KiCad schematic)
At the start: 5 parts, among them IC1 SST26VF064B-104V_MF

Commit message: Add fields to PCBA
Parts:
- C15: value 100nF -> 100n; MFN (none) -> Samsung Electro-Mechanics; MFP (none) -> CL21A106KOQNNNG; S1PL (none) -> https://www.mouser.com/ProductDetail/Samsung-Electro-Mechan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; S1PN (none) -> 187-CL21A106KOQNNNG
- IC1: Field4 SST26VF064B-104V/MF -> (none); Field5 Memory; SDI, SPI, SQI; TDFN8; 2.3÷3.6V; Memory: Serial Flas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 -> (none); Field6 WDFN-8 Microchip -> (none); Field7 Microchip -> (none); Field8 None -> (none); MFN (none) -> Microchip; MFP (none) -> SST26VF064B-104V/MF
Changed lines of the file:
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@@
       (effects (font (size 1.27 1.27)) (justify left))
     )
-    (property "Value" "100nF" (id 1) (at 177.546 78.613 0)
+    (property "Value" "100n" (id 1) (at 177.546 78.613 0)
       (effects (font (size 1.27 1.27)) (justify left))
     )
@@
     )
     (property "Datasheet" "~" (id 3) (at 174.625 77.47 0)
+      (effects (font (size 1.27 1.27)) hide)
+    )
+    (property "Description" "Multilayer Ceramic Capacitors MLCC - SMD/SMT 50V .1uF X7R 0805 10%TOL" (id 4) (at 174.625 77.47 0)
+      (effects (font (size 1.27 1.27)) hide)
+    )
+    (property "MFN" "Samsung Electro-Mechanics " (id 5) (at 174.625 77.47 0)
+      (effects (font (size 1.27 1.27)) hide)
+    )
+    (property "MFP" "CL21A106KOQNNNG " (id 6) (at 174.625 77.47 0)
+      (effects (font (size 1.27 1.27)) hide)
+    )
+    (property "S1PL" "https://www.mouser.com/ProductDetail/Samsung-Electro-Mechanics/CL21A106KOQNNNG?qs=hqM3L16%252BxlcMWI7QbqH0LA%3D%3D" (id 7) (at 174.625 77.47 0)
+      (effects (font (size 1.27 1.27)) hide)
+    )
+    (property "S1PN" " 187-CL21A106KOQNNNG " (id 8) (at 174.625 77.47 0)
       (effects (font (size 1.27 1.27)) hide)
     )
@@
       (effects (font (size 1.27 1.27)) (justify left bottom) hide)
     )
-    (property "Field4" "SST26VF064B-104V/MF" (id 4) (at 155.575 103.505 0)
+    (property "Description" "Memory; SDI, SPI, SQI; TDFN8; 2.3÷3.6V; Memory: Serial Flash; 64Mbit" (id 5) (at 155.575 103.505 0)
       (effects (font (size 1.27 1.27)) (justify left bottom) hide)
     )
-    (property "Field5" "Memory; SDI, SPI, SQI; TDFN8; 2.3÷3.6V; Memory: Serial Flash; 64Mbit" (id 5) (at 155.575 103.505 0)
-      (effects (font (size 1.27 1.27)) (justify left bottom) hide)
+    (property "MFN" "Microchip" (id 4) (at 155.575 103.505 0)
+      (effects (font (size 1.27 1.27)) hide)
     )
-    (property "Field6" "WDFN-8 Microchip" (id 6) (at 155.575 103.505 0)
-      (effects (font (size 1.27 1.27)) (justify left bottom) hide)
-    )
-    (property "Field7" "Microchip" (id 7) (at 155.575 103.505 0)
-      (effects (font (size 1.27 1.27)) (justify left bottom) hide)
-    )
-    (property "Field8" "None" (id 8) (at 155.575 103.505 0)
-      (effects (font (size 1.27 1.27)) (justify left bottom) hide)
+    (property "MFP" "SST26VF064B-104V/MF" (id 5) (at 155.575 103.505 0)
+      (effects (font (size 1.27 1.27)) hide)
     )
   )

Commit message: Update 2: Fields for BOM with PCBA manufacturer
Parts:
- IC1: value SST26VF064B-104V_MF -> SST26VF064B-104V; MFP SST26VF064B-104V/MF -> SST26VF064B-104V/SM; S1PL (none) -> https://www.mouser.com/ProductDetail/Microchip-Technology/S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; S1PN (none) -> 579-26VF064B-104V/SM
Changed lines of the file:
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@@
     (in_bom yes) (on_board yes)
     (property "Reference" "IC1" (id 0) (at 155.575 86.5632 0))
-    (property "Value" "SST26VF064B-104V_MF" (id 1) (at 155.575 88.8746 0))
+    (property "Value" "SST26VF064B-104V" (id 1) (at 155.575 88.8746 0))
     (property "Footprint" "Package_SO:SOIJ-8_5.3x5.3mm_P1.27mm" (id 2) (at 155.575 103.505 0)
       (effects (font (size 1.27 1.27)) (justify left bottom) hide)
     )
-    (property "Datasheet" "Unavailable" (id 3) (at 155.575 103.505 0)
-      (effects (font (size 1.27 1.27)) (justify left bottom) hide)
-    )
-    (property "Description" "Memory; SDI, SPI, SQI; TDFN8; 2.3÷3.6V; Memory: Serial Flash; 64Mbit" (id 5) (at 155.575 103.505 0)
+    (property "Datasheet" "http://ww1.microchip.com/downloads/en/DeviceDoc/SST26VF064B-SST26VF064BA-2.5V-3.0V-64-Mbit-Serial-Quad-IO-Flash-Memory-Data-Sheet-DS20005119J.pdf" (id 3) (at 155.575 103.505 0)
       (effects (font (size 1.27 1.27)) (justify left bottom) hide)
     )
@@
       (effects (font (size 1.27 1.27)) hide)
     )
-    (property "MFP" "SST26VF064B-104V/MF" (id 5) (at 155.575 103.505 0)
+    (property "MFP" "SST26VF064B-104V/SM" (id 4) (at 155.575 103.505 0)
       (effects (font (size 1.27 1.27)) hide)
     )
+    (property "Description" "2.5V/3.0V 64 Mbit Serial Quad I/O (SQI) Flash Memory" (id 5) (at 155.575 103.505 0)
+      (effects (font (size 1.27 1.27)) hide)
+    )
+    (property "S1PL" "https://www.mouser.com/ProductDetail/Microchip-Technology/SST26VF064B-104V-SM?qs=BA62vJVifGrueLaL24%2Fs8g%3D%3D" (id 6) (at 155.575 103.505 0)
+      (effects (font (size 1.27 1.27)) hide)
+    )
+    (property "S1PN" " 579-26VF064B-104V/SM " (id 7) (at 155.575 103.505 0)
+      (effects (font (size 1.27 1.27)) hide)
+    )

Commit message: Update 3 - BOM for PCBA
Parts:
- IC1: MFP SST26VF064B-104V/SM -> (none)
- R26: MFN (none) -> Vishay / Dale; MFP (none) -> CRCW08051K00JNEAC; S1PL (none) -> https://www.mouser.com/ProductDetail/Vishay-Dale/CRCW08051K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; S1PN (none) -> 71-CRCW08051K00JNEAC
- R27, R28: MFN (none) -> KOA Speer; MFP (none) -> RK73H2ATTD1002F; S1PL (none) -> https://www.mouser.com/ProductDetail/KOA-Speer/RK73H2ATTD10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; S1PN (none) -> 660-RK73H2ATTD1002F
Changed lines of the file:
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@@
       (effects (font (size 1.27 1.27)) hide)
     )
-    (property "Datasheet" "~" (id 3) (at 119.38 112.395 0)
+    (property "Datasheet" "https://www.mouser.com/datasheet/2/219/RK73H-1825326.pdf" (id 3) (at 119.38 112.395 0)
+      (effects (font (size 1.27 1.27)) hide)
+    )
+    (property "Description" "Thick Film Resistors - SMD 1/4W 10K OHM 1%" (id 4) (at 119.38 112.395 0)
+      (effects (font (size 1.27 1.27)) hide)
+    )
+    (property "MFN" "KOA Speer " (id 5) (at 119.38 112.395 0)
+      (effects (font (size 1.27 1.27)) hide)
+    )
+    (property "MFP" "RK73H2ATTD1002F" (id 6) (at 119.38 112.395 0)
+      (effects (font (size 1.27 1.27)) hide)
+    )
+    (property "S1PL" "https://www.mouser.com/ProductDetail/KOA-Speer/RK73H2ATTD1002F?qs=sGAEpiMZZMtlubZbdhIBIADEshVnklemK%252BhrLNEuMe8%3D" (id 7) (at 119.38 112.395 0)
+      (effects (font (size 1.27 1.27)) hide)
+    )
+    (property "S1PN" " 660-RK73H2ATTD1002F " (id 8) (at 119.38 112.395 0)
       (effects (font (size 1.27 1.27)) hide)
     )
@@
       (effects (font (size 1.27 1.27)) hide)
     )
-    (property "Datasheet" "~" (id 3) (at 130.175 106.045 0)
+    (property "Datasheet" "https://www.mouser.com/datasheet/2/219/RK73H-1825326.pdf" (id 3) (at 130.175 106.045 0)
+      (effects (font (size 1.27 1.27)) hide)
+    )
+    (property "Description" "Thick Film Resistors - SMD 1/4W 10K OHM 1%" (id 4) (at 130.175 106.045 0)
+      (effects (font (size 1.27 1.27)) hide)
+    )
+    (property "MFN" "KOA Speer " (id 5) (at 130.175 106.045 0)
+      (effects (font (size 1.27 1.27)) hide)
+    )
+    (property "MFP" "RK73H2ATTD1002F" (id 6) (at 130.175 106.045 0)
+      (effects (font (size 1.27 1.27)) hide)
+    )
+    (property "S1PL" "https://www.mouser.com/ProductDetail/KOA-Speer/RK73H2ATTD1002F?qs=sGAEpiMZZMtlubZbdhIBIADEshVnklemK%252BhrLNEuMe8%3D" (id 7) (at 130.175 106.045 0)
+      (effects (font (size 1.27 1.27)) hide)
+    )
+    (property "S1PN" " 660-RK73H2ATTD1002F " (id 8) (at 130.175 106.045 0)
       (effects (font (size 1.27 1.27)) hide)
     )
@@
       (effects (font (size 1.27 1.27)) hide)
     )
-    (property "Datasheet" "~" (id 3) (at 132.08 98.425 0)
+    (property "Datasheet" "https://www.mouser.com/datasheet/2/427/crcwce3-1762584.pdf" (id 3) (at 132.08 98.425 0)
+      (effects (font (size 1.27 1.27)) hide)
+    )
+    (property "Description" "Thick Film Resistors - SMD 1/8Watt 1Kohms 5% Commercial Use" (id 4) (at 132.08 98.425 0)
+      (effects (font (size 1.27 1.27)) hide)
+    )
+    (property "MFN" "Vishay / Dale " (id 5) (at 132.08 98.425 0)
+      (effects (font (size 1.27 1.27)) hide)
+    )
+    (property "MFP" "CRCW08051K00JNEAC " (id 6) (at 132.08 98.425 0)
+      (effects (font (size 1.27 1.27)) hide)
+    )
+    (property "S1PL" "https://www.mouser.com/ProductDetail/Vishay-Dale/CRCW08051K00JNEAC?qs=sGAEpiMZZMtlubZbdhIBIIZe04wfiaJWy7nwcSDiXks%3D" (id 7) (at 132.08 98.425 0)
+      (effects (font (size 1.27 1.27)) hide)
+    )
+    (property "S1PN" " 71-CRCW08051K00JNEAC " (id 8) (at 132.08 98.425 0)
       (effects (font (size 1.27 1.27)) hide)
     )
@@
       (effects (font (size 1.27 1.27)) hide)
     )
-    (property "MFP" "SST26VF064B-104V/SM" (id 4) (at 155.575 103.505 0)
-      (effects (font (size 1.27 1.27)) hide)
-    )

Commit message: Update 5 - BOM for PCBA. Check 1 issue #46
Parts:
- C15: MFN Samsung Electro-Mechanics -> AVX; MFP CL21A106KOQNNNG -> 08055C104KAT2A; S1PL https://www.mouser.com/ProductDetail/Samsung-Electro-Mechan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 -> https://www.mouser.com/ProductDetail/AVX/08055C104KAT2A?qs=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; S1PN 187-CL21A106KOQNNNG -> 581-08055C104K
Changed lines of the file:
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@@
       (effects (font (size 1.27 1.27)) hide)
     )
-    (property "Datasheet" "~" (id 3) (at 174.625 77.47 0)
+    (property "Datasheet" "https://www.mouser.com/datasheet/2/40/X7RDielectric-777024.pdf" (id 3) (at 174.625 77.47 0)
       (effects (font (size 1.27 1.27)) hide)
     )
@@
       (effects (font (size 1.27 1.27)) hide)
     )
-    (property "MFN" "Samsung Electro-Mechanics " (id 5) (at 174.625 77.47 0)
+    (property "MFN" "AVX " (id 5) (at 174.625 77.47 0)
       (effects (font (size 1.27 1.27)) hide)
     )
-    (property "MFP" "CL21A106KOQNNNG " (id 6) (at 174.625 77.47 0)
+    (property "MFP" "08055C104KAT2A " (id 6) (at 174.625 77.47 0)
       (effects (font (size 1.27 1.27)) hide)
     )
-    (property "S1PL" "https://www.mouser.com/ProductDetail/Samsung-Electro-Mechanics/CL21A106KOQNNNG?qs=hqM3L16%252BxlcMWI7QbqH0LA%3D%3D" (id 7) (at 174.625 77.47 0)
+    (property "S1PL" "https://www.mouser.com/ProductDetail/AVX/08055C104KAT2A?qs=2ujN4bDBNE9mJvapP%252BjopA%3D%3D" (id 7) (at 174.625 77.47 0)
       (effects (font (size 1.27 1.27)) hide)
     )
-    (property "S1PN" " 187-CL21A106KOQNNNG " (id 8) (at 174.625 77.47 0)
+    (property "S1PN" " 581-08055C104K " (id 8) (at 174.625 77.47 0)
       (effects (font (size 1.27 1.27)) hide)
     )
