File: pcb/main/Load cell 24bits ADC.kicad_sch (KiCad schematic)
At the start: 17 parts, among them J9 SJ, Q4 TRANSISTOR_PNPMMBT4403, U4 HX711

Commit message: Update 5 - BOM for PCBA. Check 1 issue #46
Parts:
- C16, C18, C19, C20: MFN Samsung Electro-Mechanics -> AVX; MFP CL21A106KOQNNNG -> 08055C104KAT2A; S1PL https://www.mouser.com/ProductDetail/Samsung-Electro-Mechan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 -> https://www.mouser.com/ProductDetail/AVX/08055C104KAT2A?qs=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; S1PN 187-CL21A106KOQNNNG -> 581-08055C104K
Changed lines of the file:
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@@
       (effects (font (size 1.27 1.27)) hide)
     )
-    (property "Datasheet" "~" (id 3) (at 96.52 123.825 0)
+    (property "Datasheet" "https://www.mouser.com/datasheet/2/40/X7RDielectric-777024.pdf" (id 3) (at 96.52 123.825 0)
       (effects (font (size 1.27 1.27)) hide)
     )
@@
       (effects (font (size 1.27 1.27)) hide)
     )
-    (property "MFN" "Samsung Electro-Mechanics " (id 5) (at 96.52 123.825 0)
+    (property "MFN" "AVX " (id 5) (at 96.52 123.825 0)
       (effects (font (size 1.27 1.27)) hide)
     )
-    (property "MFP" "CL21A106KOQNNNG " (id 6) (at 96.52 123.825 0)
+    (property "MFP" "08055C104KAT2A " (id 6) (at 96.52 123.825 0)
       (effects (font (size 1.27 1.27)) hide)
     )
-    (property "S1PL" "https://www.mouser.com/ProductDetail/Samsung-Electro-Mechanics/CL21A106KOQNNNG?qs=hqM3L16%252BxlcMWI7QbqH0LA%3D%3D" (id 7) (at 96.52 123.825 0)
+    (property "S1PL" "https://www.mouser.com/ProductDetail/AVX/08055C104KAT2A?qs=2ujN4bDBNE9mJvapP%252BjopA%3D%3D" (id 7) (at 96.52 123.825 0)
       (effects (font (size 1.27 1.27)) hide)
     )
-    (property "S1PN" " 187-CL21A106KOQNNNG " (id 8) (at 96.52 123.825 0)
+    (property "S1PN" " 581-08055C104K " (id 8) (at 96.52 123.825 0)
       (effects (font (size 1.27 1.27)) hide)
     )
@@
       (effects (font (size 1.27 1.27)) hide)
     )
-    (property "Datasheet" "~" (id 3) (at 122.555 82.55 0)
+    (property "Datasheet" "https://www.mouser.com/datasheet/2/40/X7RDielectric-777024.pdf" (id 3) (at 122.555 82.55 0)
       (effects (font (size 1.27 1.27)) hide)
     )
@@
       (effects (font (size 1.27 1.27)) hide)
     )
-    (property "MFN" "Samsung Electro-Mechanics " (id 5) (at 122.555 82.55 0)
+    (property "MFN" "AVX " (id 5) (at 122.555 82.55 0)
       (effects (font (size 1.27 1.27)) hide)
     )
-    (property "MFP" "CL21A106KOQNNNG " (id 6) (at 122.555 82.55 0)
+    (property "MFP" "08055C104KAT2A " (id 6) (at 122.555 82.55 0)
       (effects (font (size 1.27 1.27)) hide)
     )
-    (property "S1PL" "https://www.mouser.com/ProductDetail/Samsung-Electro-Mechanics/CL21A106KOQNNNG?qs=hqM3L16%252BxlcMWI7QbqH0LA%3D%3D" (id 7) (at 122.555 82.55 0)
+    (property "S1PL" "https://www.mouser.com/ProductDetail/AVX/08055C104KAT2A?qs=2ujN4bDBNE9mJvapP%252BjopA%3D%3D" (id 7) (at 122.555 82.55 0)
       (effects (font (size 1.27 1.27)) hide)
     )
-    (property "S1PN" " 187-CL21A106KOQNNNG " (id 8) (at 122.555 82.55 0)
+    (property "S1PN" " 581-08055C104K " (id 8) (at 122.555 82.55 0)
       (effects (font (size 1.27 1.27)) hide)
     )
@@
       (effects (font (size 1.27 1.27)) hide)
     )
-    (property "Datasheet" "~" (id 3) (at 147.955 104.14 0)
+    (property "Datasheet" "https://www.mouser.com/datasheet/2/40/X7RDielectric-777024.pdf" (id 3) (at 147.955 104.14 0)
       (effects (font (size 1.27 1.27)) hide)
     )
@@
       (effects (font (size 1.27 1.27)) hide)
     )
-    (property "MFN" "Samsung Electro-Mechanics " (id 5) (at 147.955 104.14 0)
+    (property "MFN" "AVX " (id 5) (at 147.955 104.14 0)
       (effects (font (size 1.27 1.27)) hide)
     )
-    (property "MFP" "CL21A106KOQNNNG " (id 6) (at 147.955 104.14 0)
+    (property "MFP" "08055C104KAT2A " (id 6) (at 147.955 104.14 0)
       (effects (font (size 1.27 1.27)) hide)
     )
-    (property "S1PL" "https://www.mouser.com/ProductDetail/Samsung-Electro-Mechanics/CL21A106KOQNNNG?qs=hqM3L16%252BxlcMWI7QbqH0LA%3D%3D" (id 7) (at 147.955 104.14 0)
+    (property "S1PL" "https://www.mouser.com/ProductDetail/AVX/08055C104KAT2A?qs=2ujN4bDBNE9mJvapP%252BjopA%3D%3D" (id 7) (at 147.955 104.14 0)
       (effects (font (size 1.27 1.27)) hide)
     )
-    (property "S1PN" " 187-CL21A106KOQNNNG " (id 8) (at 147.955 104.14 0)
+    (property "S1PN" " 581-08055C104K " (id 8) (at 147.955 104.14 0)
       (effects (font (size 1.27 1.27)) hide)
     )
@@
       (effects (font (size 1.27 1.27)) hide)
     )
-    (property "Datasheet" "~" (id 3) (at 150.495 93.98 0)
+    (property "Datasheet" "https://www.mouser.com/datasheet/2/40/X7RDielectric-777024.pdf" (id 3) (at 150.495 93.98 0)
       (effects (font (size 1.27 1.27)) hide)
     )
@@
       (effects (font (size 1.27 1.27)) hide)
     )
-    (property "MFN" "Samsung Electro-Mechanics " (id 5) (at 150.495 93.98 0)
+    (property "MFN" "AVX " (id 5) (at 150.495 93.98 0)
       (effects (font (size 1.27 1.27)) hide)
     )
-    (property "MFP" "CL21A106KOQNNNG " (id 6) (at 150.495 93.98 0)
+    (property "MFP" "08055C104KAT2A " (id 6) (at 150.495 93.98 0)
       (effects (font (size 1.27 1.27)) hide)
     )
-    (property "S1PL" "https://www.mouser.com/ProductDetail/Samsung-Electro-Mechanics/CL21A106KOQNNNG?qs=hqM3L16%252BxlcMWI7QbqH0LA%3D%3D" (id 7) (at 150.495 93.98 0)
+    (property "S1PL" "https://www.mouser.com/ProductDetail/AVX/08055C104KAT2A?qs=2ujN4bDBNE9mJvapP%252BjopA%3D%3D" (id 7) (at 150.495 93.98 0)
       (effects (font (size 1.27 1.27)) hide)
     )
-    (property "S1PN" " 187-CL21A106KOQNNNG " (id 8) (at 150.495 93.98 0)
+    (property "S1PN" " 581-08055C104K " (id 8) (at 150.495 93.98 0)
       (effects (font (size 1.27 1.27)) hide)
     )
