File: pcb/main/Stepper.kicad_sch (KiCad schematic)
At the start: 38 parts, among them IC2 DRV8811, J10 SJ, J11 SJ

Commit message: Add fields to PCBA
Parts:
- C22, C23, C26: value 220nF -> 220n
- C24, C27, C28, C29, C32, C33: value 100nF -> 100n; MFN (none) -> Samsung Electro-Mechanics; MFP (none) -> CL21A106KOQNNNG; S1PL (none) -> https://www.mouser.com/ProductDetail/Samsung-Electro-Mechan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; S1PN (none) -> 187-CL21A106KOQNNNG
- C25: value 100uF 50V -> 100u
- C30, C31: value 1nF -> 1n
- C36, C37: MFN (none) -> Samsung Electro-Mechanics; MFP (none) -> CL21A106KOQNNNG; S1PL (none) -> https://www.mouser.com/ProductDetail/Samsung-Electro-Mechan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; S1PN (none) -> 187-CL21A106KOQNNNG
- R43, R44: value 0.1R 1W -> 0.1
Other:
- note added: "1 W 2010"
- note added: "50 V"
- note removed: "2010"

Commit message: Update 2: Fields for BOM with PCBA manufacturer
Parts:
- C22, C23, C26: MFN (none) -> Samsung Electro-Mechanics; MFP (none) -> CL21B224KAFNNNE; S1PL (none) -> https://www.mouser.com/ProductDetail/Samsung-Electro-Mechan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; S1PN (none) -> 187-CL21B224KAFNNNE
- C30, C31: MFN (none) -> Wurth Elektronik; MFP (none) -> 885012207060; S1PL (none) -> https://www.mouser.com/ProductDetail/Wurth-Elektronik/88501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; S1PN (none) -> 710-885012207060
- D14, D15, D16, D17: MFN (none) -> Wurth Elektronik; MFP (none) -> 150080SS75000; S1PL (none) -> https://www.mouser.com/ProductDetail/Wurth-Elektronik/15008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; S1PN (none) -> 710-150080SS75000
- IC2: MFN (none) -> Texas Instruments; MFP (none) -> DRV8811PWPR; S1PL (none) -> https://www.mouser.com/ProductDetail/Texas-Instruments/DRV8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; S1PN (none) -> 595-DRV8811PWPR
- JP10, JP11, JP12, JP7: MFN (none) -> Molex; MFP (none) -> 22-28-4040; S1PL (none) -> https://www.mouser.com/ProductDetail/Molex/22-28-4040?qs=Mu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; S1PN (none) -> 538-22-28-4040

Commit message: Update 3 - BOM for PCBA
Parts:
- C25: MFN (none) -> Lelon; MFP (none) -> VZL101M1ETR-0607; S1PL (none) -> https://www.mouser.com/ProductDetail/Lelon/VZL101M1ETR-0607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; S1PN (none) -> 140-VZL101M1ETR-0607
- R34, R36, R39, R40, R42, R49: MFN (none) -> KOA Speer; MFP (none) -> RK73H2ATTD1002F; S1PL (none) -> https://www.mouser.com/ProductDetail/KOA-Speer/RK73H2ATTD10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; S1PN (none) -> 660-RK73H2ATTD1002F
- R41: MFN (none) -> KOA Speer; MFP (none) -> RK73H2ATTD3301F; S1PL (none) -> https://www.mouser.com/ProductDetail/KOA-Speer/RK73H2ATTD33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; S1PN (none) -> 660-RK73H2ATTD3301F
- R43, R44: MFN (none) -> IRC / TT Electronics; MFP (none) -> LRC-LR2010LF-01-R100-F; S1PL (none) -> https://www.mouser.com/ProductDetail/IRC-TT-Electronics/LRC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; S1PN (none) -> 66-LR2010LF-01-R100
- R45, R46, R48: MFN (none) -> KOA Speer; MFP (none) -> RK73H2ATTD4702F; S1PL (none) -> https://www.mouser.com/ProductDetail/KOA-Speer/RK73H2ATTD47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; S1PN (none) -> 660-RK73H2ATTD4702F

Commit message: Update 5 - BOM for PCBA. Check 1 issue #46
Parts:
- C24, C27, C28, C29, C32, C33, C36, C37: MFN Samsung Electro-Mechanics -> AVX; MFP CL21A106KOQNNNG -> 08055C104KAT2A; S1PL https://www.mouser.com/ProductDetail/Samsung-Electro-Mechan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 -> https://www.mouser.com/ProductDetail/AVX/08055C104KAT2A?qs=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; S1PN 187-CL21A106KOQNNNG -> 581-08055C104K
- R47: value Rlim -> 180; MFN (none) -> KOA Speer; MFP (none) -> RK73H2ATTD1800F; S1PL (none) -> https://www.mouser.com/ProductDetail/KOA-Speer/RK73H2ATTD18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; S1PN (none) -> 660-RK73H2ATTD1800F
Other:
- note added: "Rlim Approx. 180 Ohms"
